File: hardware/octoprobe_kicad_v1/pcb_dezentral.kicad_pcb (KiCad board)
At the start: 2 copper layers, 55 x 73.5 mm, 98 parts, among them J1 weidmueller_SL5.08HC-06-90, J2 weidmueller_SL5.08HC-10-90, J901 USB_C_Receptacle_USB2.0, Q1 AO3400A, SW1 dip_switch_SPST16, SW901 SW_MEC_5E, U1 SP3485EN-L/TR, U2 AOZ1282CI, U901 RP2040, U902 AMS1117-3.3, U903 W25Q128JVS, Y901 Crystal_GND24_Small

Commit message: cleanup pcb
Parts:
- removed C1: 4u7 50V, Diode_SMD:D_1206_3216Metric
- removed C2, C3, C5, C6, C7: 100n 50V, Diode_SMD:D_0805_2012Metric
- removed C4: 10u 25V, Diode_SMD:D_0805_2012Metric
- removed D1, D10, D11, D12, D13, D14, D15, D16, D19, D2, D20, D24, D25, D3, D4, D5, D6, D7, D8, D9: B5819W SL, Diode_SMD:D_SOD-123
- removed D17: LED RED, 00_project_library:LED_0603_1608Metric
- removed D18: LED WHITE, 00_project_library:LED_0603_1608Metric
- removed D21, D22, D23: SMBJ6.5CA, Diode_SMD:D_SMB
- removed D26: SMBJ30CA, Diode_SMD:D_SMB
- removed D27: LED BLUE, 00_project_library:LED_0603_1608Metric
- removed HOLDER1: ~, 00_project_library:din_rail_pcb_holder
- removed J1: weidmueller_SL5.08HC-06-90, 00_project_library:weidmueller_SL5.08HC-06-90
- removed J2: weidmueller_SL5.08HC-10-90, 00_project_library:weidmueller_SL5.08HC-10-90
- removed L1: 22uH, 00_project_library:L_MODBUS
- removed Q1: AO3400A, Package_TO_SOT_SMD:SOT-23
- removed R1, R14, R17, R2, R3, R4, R5, R6, R7, R8: 4k7, Resistor_SMD:R_0402_1005Metric_Pad0.72x0.64mm_HandSolder
- removed R10, R13, R18, R19: 10k, Resistor_SMD:R_0402_1005Metric_Pad0.72x0.64mm_HandSolder
- removed R11: 100k, Resistor_SMD:R_0402_1005Metric_Pad0.72x0.64mm_HandSolder
- removed R12: 56k, Resistor_SMD:R_0402_1005Metric_Pad0.72x0.64mm_HandSolder
- removed R15, R16: 470R, Resistor_SMD:R_0402_1005Metric_Pad0.72x0.64mm_HandSolder
- removed R9: 470, Resistor_SMD:R_0402_1005Metric_Pad0.72x0.64mm_HandSolder
- removed SW1: dip_switch_SPST16, 00_project_library:dip_switch_SPST16
- removed U1: SP3485EN-L/TR, Package_SO:SOIC-8_3.9x4.9mm_P1.27mm
- removed U2: AOZ1282CI, Package_TO_SOT_SMD:SOT-23-6
Routing:
- net +3V3: track 283.6 -> 92.3 mm, vias 2 -> 0
- net ds_7: track 74.3 -> 0.00 mm
- net ds_6: track 70.3 -> 0.00 mm
- net ds_5: track 66.5 -> 0.00 mm
- net ds_4: track 62.5 -> 0.00 mm
- net ds_3: track 58.2 -> 0.00 mm
- net ds_2: track 53.8 -> 0.00 mm
- net GND: track 100.8 -> 50.6 mm, vias 42 -> 19
- net ds_1: track 50.1 -> 0.00 mm
- net +5V: track 60.2 -> 10.5 mm
- net ds_0: track 48.2 -> 0.00 mm
- net rel: track 44.2 -> 0.00 mm, vias 3 -> 0
- net MODBUS_RO: track 41.0 -> 0.00 mm, vias 4 -> 0
- net MODBUS_DE: track 40.1 -> 0.00 mm, vias 2 -> 0
- net 485_D+: track 39.8 -> 0.00 mm
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Other:
- board text removed: "*"
- board text removed: "0V"
- board text removed: "24V"
- board text removed: "3V3"
- board text removed: "485"
- board text removed: "D+"
- board text removed: "D-"
- board text removed: "DS_1"
- board text removed: "DS_2"
- board text removed: "DS_3"
- board text removed: "DS_4"
- board text removed: "DS_5"
- board text removed: "DS_6"
- board text removed: "DS_7"
- board text removed: "GND"
- board text removed: "MODBUS"
- board text removed: "RX"
- board text removed: "TX"
- board text removed: "locked"
- board text removed: "rel_n"
- board text removed: "rel_p"

Commit message: initial
Parts:
- added C101: 100n 50V, Diode_SMD:D_0805_2012Metric, F.Cu at (50.8, 96.2)
- added D1001: LED WHITE, 00_project_library:LED_0603_1608Metric, F.Cu at (162.6, 85.6)
- added D301: LED WHITE, 00_project_library:LED_0603_1608Metric, F.Cu at (122.0, 85.6)
- added D401: LED WHITE, 00_project_library:LED_0603_1608Metric, F.Cu at (132.2, 85.6)
- added D501: RED, 00_project_library:LED_0603_1608Metric, F.Cu at (101.7, 85.6)
- added D601: RED, 00_project_library:LED_0603_1608Metric, F.Cu at (111.8, 85.6)
- added D701: LED WHITE, 00_project_library:LED_0603_1608Metric, F.Cu at (142.4, 85.6)
- added D901: LED WHITE, 00_project_library:LED_0603_1608Metric, F.Cu at (152.4, 85.6)
- added FanQ501: NMOS, Package_TO_SOT_SMD:SOT-23, F.Cu at (102.1, 94.2)
- added FanQ601: NMOS, Package_TO_SOT_SMD:SOT-23, F.Cu at (112.2, 94.2)
- added J1001: Conn_01x02_Socket, Connector_PinSocket_2.54mm:PinSocket_1x02_P2.54mm_Vertical, F.Cu at (161.4, 98.8)
- added J1002: Conn_01x02_Socket, Connector_PinSocket_2.54mm:PinSocket_1x02_P2.54mm_Vertical, F.Cu at (161.4, 102.6)
- added J1003: Conn_01x02_Pin, Connector_PinHeader_2.54mm:PinHeader_1x02_P2.54mm_Vertical, F.Cu at (163.9, 106.4)
- added J101: Conn_01x20, 00_project_library:PinSocket_2x20_P2.54mm_Vertical-stackable, F.Cu at (165.4, 129.0)
- added J102: Conn_01x20, 00_project_library:PinSocket_2x20_P2.54mm_Vertical-mirrored, F.Cu at (157.8, 129.0)
- added J103: Conn_01x20, 00_project_library:PinSocket_2x20_P2.54mm_Vertical-mirrored-bare, F.Cu at (150.2, 129.0)
- added J301: Conn_01x02_Socket, Connector_PinSocket_2.54mm:PinSocket_1x02_P2.54mm_Vertical, F.Cu at (120.8, 98.8)
- added J302: Conn_01x02_Socket, Connector_PinSocket_2.54mm:PinSocket_1x02_P2.54mm_Vertical, F.Cu at (120.8, 102.6)
- added J303: Conn_01x02_Pin, Connector_PinHeader_2.54mm:PinHeader_1x02_P2.54mm_Vertical, F.Cu at (123.3, 106.4)
- added J401: Conn_01x02_Socket, Connector_PinSocket_2.54mm:PinSocket_1x02_P2.54mm_Vertical, F.Cu at (131.0, 98.8)
- added J402: Conn_01x02_Socket, Connector_PinSocket_2.54mm:PinSocket_1x02_P2.54mm_Vertical, F.Cu at (131.0, 102.6)
- added J403: Conn_01x02_Pin, Connector_PinHeader_2.54mm:PinHeader_1x02_P2.54mm_Vertical, F.Cu at (133.5, 106.4)
- added J501: Conn_01x02_Socket, Connector_PinSocket_2.54mm:PinSocket_1x02_P2.54mm_Vertical, F.Cu at (100.9, 102.6)
- added J502: Conn_01x02_Socket, Connector_PinSocket_2.54mm:PinSocket_1x02_P2.54mm_Vertical, F.Cu at (100.9, 98.8)
- added J503: Conn_01x02_Pin, Connector_PinHeader_2.54mm:PinHeader_1x02_P2.54mm_Vertical, F.Cu at (103.5, 106.4)
- added J601: Conn_01x02_Socket, Connector_PinSocket_2.54mm:PinSocket_1x02_P2.54mm_Vertical, F.Cu at (111.1, 102.6)
- added J602: Conn_01x02_Socket, Connector_PinSocket_2.54mm:PinSocket_1x02_P2.54mm_Vertical, F.Cu at (111.1, 98.8)
- added J603: Conn_01x02_Pin, Connector_PinHeader_2.54mm:PinHeader_1x02_P2.54mm_Vertical, F.Cu at (113.6, 106.4)
- added J701: Conn_01x02_Socket, Connector_PinSocket_2.54mm:PinSocket_1x02_P2.54mm_Vertical, F.Cu at (141.2, 98.8)
- added J702: Conn_01x02_Socket, Connector_PinSocket_2.54mm:PinSocket_1x02_P2.54mm_Vertical, F.Cu at (141.2, 102.6)
- added J703: Conn_01x02_Pin, Connector_PinHeader_2.54mm:PinHeader_1x02_P2.54mm_Vertical, F.Cu at (143.7, 106.4)
- added J801: Conn_01x02_Socket, Connector_PinSocket_2.54mm:PinSocket_1x02_P2.54mm_Vertical, F.Cu at (90.8, 102.6)
- added J802: Conn_01x02_Socket, Connector_PinSocket_2.54mm:PinSocket_1x02_P2.54mm_Vertical, F.Cu at (90.8, 98.8)
- added J803: Conn_01x02_Pin, Connector_PinHeader_2.54mm:PinHeader_1x02_P2.54mm_Vertical, F.Cu at (93.4, 106.4)
- added J901: Conn_01x02_Socket, Connector_PinSocket_2.54mm:PinSocket_1x02_P2.54mm_Vertical, F.Cu at (151.2, 98.8)
- added J902: Conn_01x02_Socket, Connector_PinSocket_2.54mm:PinSocket_1x02_P2.54mm_Vertical, F.Cu at (151.2, 102.6)
- added J903: Conn_01x02_Pin, Connector_PinHeader_2.54mm:PinHeader_1x02_P2.54mm_Vertical, F.Cu at (153.8, 106.4)
- added R1001: 1k, Resistor_SMD:R_0402_1005Metric_Pad0.72x0.64mm_HandSolder, F.Cu at (160.3, 89.9)
- added R1002: 10K, Resistor_SMD:R_0402_1005Metric_Pad0.72x0.64mm_HandSolder, F.Cu at (164.9, 89.9)
- added R301: 1k, Resistor_SMD:R_0402_1005Metric_Pad0.72x0.64mm_HandSolder, F.Cu at (119.7, 89.9)
- added R302: 10K, Resistor_SMD:R_0402_1005Metric_Pad0.72x0.64mm_HandSolder, F.Cu at (124.3, 89.9)
- added R401: 1k, Resistor_SMD:R_0402_1005Metric_Pad0.72x0.64mm_HandSolder, F.Cu at (129.9, 89.9)
- added R402: 10K, Resistor_SMD:R_0402_1005Metric_Pad0.72x0.64mm_HandSolder, F.Cu at (134.5, 89.9)
- added R501: 470R, Resistor_SMD:R_0402_1005Metric_Pad0.72x0.64mm_HandSolder, F.Cu at (101.3, 90.2)
- added R601: 470R, Resistor_SMD:R_0402_1005Metric_Pad0.72x0.64mm_HandSolder, F.Cu at (111.4, 90.2)
- added R701: 1k, Resistor_SMD:R_0402_1005Metric_Pad0.72x0.64mm_HandSolder, F.Cu at (140.1, 89.9)
- added R702: 10K, Resistor_SMD:R_0402_1005Metric_Pad0.72x0.64mm_HandSolder, F.Cu at (144.7, 89.9)
- added R901: 1k, Resistor_SMD:R_0402_1005Metric_Pad0.72x0.64mm_HandSolder, F.Cu at (150.2, 89.9)
- added R902: 10K, Resistor_SMD:R_0402_1005Metric_Pad0.72x0.64mm_HandSolder, F.Cu at (154.7, 89.9)
- added REF**: MountingHole_4.3mm_M4, MountingHole:MountingHole_4.3mm_M4, F.Cu at (166.5, 40.0)
- added REF**: MountingHole_4.3mm_M4, MountingHole:MountingHole_4.3mm_M4, F.Cu at (166.5, 185.0)
- added REF**: MountingHole_4.3mm_M4, MountingHole:MountingHole_4.3mm_M4, F.Cu at (81.5, 40.0)
- added REF**: MountingHole_4.3mm_M4, MountingHole:MountingHole_4.3mm_M4, F.Cu at (81.5, 185.0)
- added REF**: TestPoint_THTPad_D2.0mm_Drill1.0mm, TestPoint:TestPoint_THTPad_D2.0mm_Drill1.0mm, F.Cu at (79.1, 129.0)
- added REF**1: TestPoint_THTPad_D2.0mm_Drill1.0mm, TestPoint:TestPoint_THTPad_D2.0mm_Drill1.0mm, F.Cu at (81.6, 129.0)
- added REF**10: TestPoint_THTPad_D2.0mm_Drill1.0mm, TestPoint:TestPoint_THTPad_D2.0mm_Drill1.0mm, F.Cu at (104.5, 129.0)
- added REF**100: TestPoint_THTPad_D2.0mm_Drill1.0mm, TestPoint:TestPoint_THTPad_D2.0mm_Drill1.0mm, F.Cu at (135.0, 136.6)
- added REF**101: TestPoint_THTPad_D2.0mm_Drill1.0mm, TestPoint:TestPoint_THTPad_D2.0mm_Drill1.0mm, F.Cu at (137.5, 136.6)
- added REF**102: TestPoint_THTPad_D2.0mm_Drill1.0mm, TestPoint:TestPoint_THTPad_D2.0mm_Drill1.0mm, F.Cu at (140.0, 136.6)
- added REF**103: TestPoint_THTPad_D2.0mm_Drill1.0mm, TestPoint:TestPoint_THTPad_D2.0mm_Drill1.0mm, F.Cu at (142.6, 136.6)
- added REF**104: TestPoint_THTPad_D2.0mm_Drill1.0mm, TestPoint:TestPoint_THTPad_D2.0mm_Drill1.0mm, F.Cu at (79.1, 139.2)
- added REF**105: TestPoint_THTPad_D2.0mm_Drill1.0mm, TestPoint:TestPoint_THTPad_D2.0mm_Drill1.0mm, F.Cu at (81.6, 139.2)
- added REF**106: TestPoint_THTPad_D2.0mm_Drill1.0mm, TestPoint:TestPoint_THTPad_D2.0mm_Drill1.0mm, F.Cu at (84.2, 139.2)
- added REF**107: TestPoint_THTPad_D2.0mm_Drill1.0mm, TestPoint:TestPoint_THTPad_D2.0mm_Drill1.0mm, F.Cu at (86.7, 139.2)
- added REF**108: TestPoint_THTPad_D2.0mm_Drill1.0mm, TestPoint:TestPoint_THTPad_D2.0mm_Drill1.0mm, F.Cu at (89.2, 139.2)
- added REF**109: TestPoint_THTPad_D2.0mm_Drill1.0mm, TestPoint:TestPoint_THTPad_D2.0mm_Drill1.0mm, F.Cu at (91.8, 139.2)
- added REF**11: TestPoint_THTPad_D2.0mm_Drill1.0mm, TestPoint:TestPoint_THTPad_D2.0mm_Drill1.0mm, F.Cu at (107.0, 129.0)
- added REF**110: TestPoint_THTPad_D2.0mm_Drill1.0mm, TestPoint:TestPoint_THTPad_D2.0mm_Drill1.0mm, F.Cu at (94.3, 139.2)
- added REF**111: TestPoint_THTPad_D2.0mm_Drill1.0mm, TestPoint:TestPoint_THTPad_D2.0mm_Drill1.0mm, F.Cu at (96.9, 139.2)
- added REF**112: TestPoint_THTPad_D2.0mm_Drill1.0mm, TestPoint:TestPoint_THTPad_D2.0mm_Drill1.0mm, F.Cu at (99.4, 139.2)
- added REF**113: TestPoint_THTPad_D2.0mm_Drill1.0mm, TestPoint:TestPoint_THTPad_D2.0mm_Drill1.0mm, F.Cu at (101.9, 139.2)
- added REF**114: TestPoint_THTPad_D2.0mm_Drill1.0mm, TestPoint:TestPoint_THTPad_D2.0mm_Drill1.0mm, F.Cu at (104.5, 139.2)
- added REF**115: TestPoint_THTPad_D2.0mm_Drill1.0mm, TestPoint:TestPoint_THTPad_D2.0mm_Drill1.0mm, F.Cu at (107.0, 139.2)
- added REF**116: TestPoint_THTPad_D2.0mm_Drill1.0mm, TestPoint:TestPoint_THTPad_D2.0mm_Drill1.0mm, F.Cu at (109.6, 139.2)
- added REF**117: TestPoint_THTPad_D2.0mm_Drill1.0mm, TestPoint:TestPoint_THTPad_D2.0mm_Drill1.0mm, F.Cu at (112.1, 139.2)
- added REF**118: TestPoint_THTPad_D2.0mm_Drill1.0mm, TestPoint:TestPoint_THTPad_D2.0mm_Drill1.0mm, F.Cu at (114.6, 139.2)
- added REF**119: TestPoint_THTPad_D2.0mm_Drill1.0mm, TestPoint:TestPoint_THTPad_D2.0mm_Drill1.0mm, F.Cu at (117.2, 139.2)
- added REF**12: TestPoint_THTPad_D2.0mm_Drill1.0mm, TestPoint:TestPoint_THTPad_D2.0mm_Drill1.0mm, F.Cu at (109.6, 129.0)
- added REF**120: TestPoint_THTPad_D2.0mm_Drill1.0mm, TestPoint:TestPoint_THTPad_D2.0mm_Drill1.0mm, F.Cu at (119.7, 139.2)
- added REF**121: TestPoint_THTPad_D2.0mm_Drill1.0mm, TestPoint:TestPoint_THTPad_D2.0mm_Drill1.0mm, F.Cu at (122.3, 139.2)
- added REF**122: TestPoint_THTPad_D2.0mm_Drill1.0mm, TestPoint:TestPoint_THTPad_D2.0mm_Drill1.0mm, F.Cu at (124.8, 139.2)
- added REF**123: TestPoint_THTPad_D2.0mm_Drill1.0mm, TestPoint:TestPoint_THTPad_D2.0mm_Drill1.0mm, F.Cu at (127.3, 139.2)
- added REF**124: TestPoint_THTPad_D2.0mm_Drill1.0mm, TestPoint:TestPoint_THTPad_D2.0mm_Drill1.0mm, F.Cu at (129.9, 139.2)
- added REF**125: TestPoint_THTPad_D2.0mm_Drill1.0mm, TestPoint:TestPoint_THTPad_D2.0mm_Drill1.0mm, F.Cu at (132.4, 139.2)
- added REF**126: TestPoint_THTPad_D2.0mm_Drill1.0mm, TestPoint:TestPoint_THTPad_D2.0mm_Drill1.0mm, F.Cu at (135.0, 139.2)
- added REF**127: TestPoint_THTPad_D2.0mm_Drill1.0mm, TestPoint:TestPoint_THTPad_D2.0mm_Drill1.0mm, F.Cu at (137.5, 139.2)
- added REF**128: TestPoint_THTPad_D2.0mm_Drill1.0mm, TestPoint:TestPoint_THTPad_D2.0mm_Drill1.0mm, F.Cu at (140.0, 139.2)
- added REF**129: TestPoint_THTPad_D2.0mm_Drill1.0mm, TestPoint:TestPoint_THTPad_D2.0mm_Drill1.0mm, F.Cu at (142.6, 139.2)
- added REF**13: TestPoint_THTPad_D2.0mm_Drill1.0mm, TestPoint:TestPoint_THTPad_D2.0mm_Drill1.0mm, F.Cu at (112.1, 129.0)
- added REF**130: TestPoint_THTPad_D2.0mm_Drill1.0mm, TestPoint:TestPoint_THTPad_D2.0mm_Drill1.0mm, F.Cu at (79.1, 141.7)
- added REF**131: TestPoint_THTPad_D2.0mm_Drill1.0mm, TestPoint:TestPoint_THTPad_D2.0mm_Drill1.0mm, F.Cu at (81.6, 141.7)
- added REF**132: TestPoint_THTPad_D2.0mm_Drill1.0mm, TestPoint:TestPoint_THTPad_D2.0mm_Drill1.0mm, F.Cu at (84.2, 141.7)
- added REF**133: TestPoint_THTPad_D2.0mm_Drill1.0mm, TestPoint:TestPoint_THTPad_D2.0mm_Drill1.0mm, F.Cu at (86.7, 141.7)
- added REF**134: TestPoint_THTPad_D2.0mm_Drill1.0mm, TestPoint:TestPoint_THTPad_D2.0mm_Drill1.0mm, F.Cu at (89.2, 141.7)
- added REF**135: TestPoint_THTPad_D2.0mm_Drill1.0mm, TestPoint:TestPoint_THTPad_D2.0mm_Drill1.0mm, F.Cu at (91.8, 141.7)
- added REF**136: TestPoint_THTPad_D2.0mm_Drill1.0mm, TestPoint:TestPoint_THTPad_D2.0mm_Drill1.0mm, F.Cu at (94.3, 141.7)
- added REF**137: TestPoint_THTPad_D2.0mm_Drill1.0mm, TestPoint:TestPoint_THTPad_D2.0mm_Drill1.0mm, F.Cu at (96.9, 141.7)
- added REF**138: TestPoint_THTPad_D2.0mm_Drill1.0mm, TestPoint:TestPoint_THTPad_D2.0mm_Drill1.0mm, F.Cu at (99.4, 141.7)
- added REF**139: TestPoint_THTPad_D2.0mm_Drill1.0mm, TestPoint:TestPoint_THTPad_D2.0mm_Drill1.0mm, F.Cu at (101.9, 141.7)
- added REF**14: TestPoint_THTPad_D2.0mm_Drill1.0mm, TestPoint:TestPoint_THTPad_D2.0mm_Drill1.0mm, F.Cu at (114.6, 129.0)
- added REF**140: TestPoint_THTPad_D2.0mm_Drill1.0mm, TestPoint:TestPoint_THTPad_D2.0mm_Drill1.0mm, F.Cu at (104.5, 141.7)
- added REF**141: TestPoint_THTPad_D2.0mm_Drill1.0mm, TestPoint:TestPoint_THTPad_D2.0mm_Drill1.0mm, F.Cu at (107.0, 141.7)
- added REF**142: TestPoint_THTPad_D2.0mm_Drill1.0mm, TestPoint:TestPoint_THTPad_D2.0mm_Drill1.0mm, F.Cu at (109.6, 141.7)
- added REF**143: TestPoint_THTPad_D2.0mm_Drill1.0mm, TestPoint:TestPoint_THTPad_D2.0mm_Drill1.0mm, F.Cu at (112.1, 141.7)
- added REF**144: TestPoint_THTPad_D2.0mm_Drill1.0mm, TestPoint:TestPoint_THTPad_D2.0mm_Drill1.0mm, F.Cu at (114.6, 141.7)
- added REF**145: TestPoint_THTPad_D2.0mm_Drill1.0mm, TestPoint:TestPoint_THTPad_D2.0mm_Drill1.0mm, F.Cu at (117.2, 141.7)
- added REF**146: TestPoint_THTPad_D2.0mm_Drill1.0mm, TestPoint:TestPoint_THTPad_D2.0mm_Drill1.0mm, F.Cu at (119.7, 141.7)
- added REF**147: TestPoint_THTPad_D2.0mm_Drill1.0mm, TestPoint:TestPoint_THTPad_D2.0mm_Drill1.0mm, F.Cu at (122.3, 141.7)
- added REF**148: TestPoint_THTPad_D2.0mm_Drill1.0mm, TestPoint:TestPoint_THTPad_D2.0mm_Drill1.0mm, F.Cu at (124.8, 141.7)
- added REF**149: TestPoint_THTPad_D2.0mm_Drill1.0mm, TestPoint:TestPoint_THTPad_D2.0mm_Drill1.0mm, F.Cu at (127.3, 141.7)
- added REF**15: TestPoint_THTPad_D2.0mm_Drill1.0mm, TestPoint:TestPoint_THTPad_D2.0mm_Drill1.0mm, F.Cu at (117.2, 129.0)
- added REF**150: TestPoint_THTPad_D2.0mm_Drill1.0mm, TestPoint:TestPoint_THTPad_D2.0mm_Drill1.0mm, F.Cu at (129.9, 141.7)
- added REF**151: TestPoint_THTPad_D2.0mm_Drill1.0mm, TestPoint:TestPoint_THTPad_D2.0mm_Drill1.0mm, F.Cu at (132.4, 141.7)
- added REF**152: TestPoint_THTPad_D2.0mm_Drill1.0mm, TestPoint:TestPoint_THTPad_D2.0mm_Drill1.0mm, F.Cu at (135.0, 141.7)
- added REF**153: TestPoint_THTPad_D2.0mm_Drill1.0mm, TestPoint:TestPoint_THTPad_D2.0mm_Drill1.0mm, F.Cu at (137.5, 141.7)
- added REF**154: TestPoint_THTPad_D2.0mm_Drill1.0mm, TestPoint:TestPoint_THTPad_D2.0mm_Drill1.0mm, F.Cu at (140.0, 141.7)
- added REF**155: TestPoint_THTPad_D2.0mm_Drill1.0mm, TestPoint:TestPoint_THTPad_D2.0mm_Drill1.0mm, F.Cu at (142.6, 141.7)
- added REF**156: TestPoint_THTPad_D2.0mm_Drill1.0mm, TestPoint:TestPoint_THTPad_D2.0mm_Drill1.0mm, F.Cu at (79.1, 144.3)
- added REF**157: TestPoint_THTPad_D2.0mm_Drill1.0mm, TestPoint:TestPoint_THTPad_D2.0mm_Drill1.0mm, F.Cu at (81.6, 144.3)
- added REF**158: TestPoint_THTPad_D2.0mm_Drill1.0mm, TestPoint:TestPoint_THTPad_D2.0mm_Drill1.0mm, F.Cu at (84.2, 144.3)
- added REF**159: TestPoint_THTPad_D2.0mm_Drill1.0mm, TestPoint:TestPoint_THTPad_D2.0mm_Drill1.0mm, F.Cu at (86.7, 144.3)
- added REF**16: TestPoint_THTPad_D2.0mm_Drill1.0mm, TestPoint:TestPoint_THTPad_D2.0mm_Drill1.0mm, F.Cu at (119.7, 129.0)
- added REF**160: TestPoint_THTPad_D2.0mm_Drill1.0mm, TestPoint:TestPoint_THTPad_D2.0mm_Drill1.0mm, F.Cu at (89.2, 144.3)
- added REF**161: TestPoint_THTPad_D2.0mm_Drill1.0mm, TestPoint:TestPoint_THTPad_D2.0mm_Drill1.0mm, F.Cu at (91.8, 144.3)
- added REF**162: TestPoint_THTPad_D2.0mm_Drill1.0mm, TestPoint:TestPoint_THTPad_D2.0mm_Drill1.0mm, F.Cu at (94.3, 144.3)
- added REF**163: TestPoint_THTPad_D2.0mm_Drill1.0mm, TestPoint:TestPoint_THTPad_D2.0mm_Drill1.0mm, F.Cu at (96.9, 144.3)
- added REF**164: TestPoint_THTPad_D2.0mm_Drill1.0mm, TestPoint:TestPoint_THTPad_D2.0mm_Drill1.0mm, F.Cu at (99.4, 144.3)
- added REF**165: TestPoint_THTPad_D2.0mm_Drill1.0mm, TestPoint:TestPoint_THTPad_D2.0mm_Drill1.0mm, F.Cu at (101.9, 144.3)
- added REF**166: TestPoint_THTPad_D2.0mm_Drill1.0mm, TestPoint:TestPoint_THTPad_D2.0mm_Drill1.0mm, F.Cu at (104.5, 144.3)
- added REF**167: TestPoint_THTPad_D2.0mm_Drill1.0mm, TestPoint:TestPoint_THTPad_D2.0mm_Drill1.0mm, F.Cu at (107.0, 144.3)
- added REF**168: TestPoint_THTPad_D2.0mm_Drill1.0mm, TestPoint:TestPoint_THTPad_D2.0mm_Drill1.0mm, F.Cu at (109.6, 144.3)
- added REF**169: TestPoint_THTPad_D2.0mm_Drill1.0mm, TestPoint:TestPoint_THTPad_D2.0mm_Drill1.0mm, F.Cu at (112.1, 144.3)
- added REF**17: TestPoint_THTPad_D2.0mm_Drill1.0mm, TestPoint:TestPoint_THTPad_D2.0mm_Drill1.0mm, F.Cu at (122.3, 129.0)
- added REF**170: TestPoint_THTPad_D2.0mm_Drill1.0mm, TestPoint:TestPoint_THTPad_D2.0mm_Drill1.0mm, F.Cu at (114.6, 144.3)
- added REF**171: TestPoint_THTPad_D2.0mm_Drill1.0mm, TestPoint:TestPoint_THTPad_D2.0mm_Drill1.0mm, F.Cu at (117.2, 144.3)
- added REF**172: TestPoint_THTPad_D2.0mm_Drill1.0mm, TestPoint:TestPoint_THTPad_D2.0mm_Drill1.0mm, F.Cu at (119.7, 144.3)
- added REF**173: TestPoint_THTPad_D2.0mm_Drill1.0mm, TestPoint:TestPoint_THTPad_D2.0mm_Drill1.0mm, F.Cu at (122.3, 144.3)
- added REF**174: TestPoint_THTPad_D2.0mm_Drill1.0mm, TestPoint:TestPoint_THTPad_D2.0mm_Drill1.0mm, F.Cu at (124.8, 144.3)
- added REF**175: TestPoint_THTPad_D2.0mm_Drill1.0mm, TestPoint:TestPoint_THTPad_D2.0mm_Drill1.0mm, F.Cu at (127.3, 144.3)
- added REF**176: TestPoint_THTPad_D2.0mm_Drill1.0mm, TestPoint:TestPoint_THTPad_D2.0mm_Drill1.0mm, F.Cu at (129.9, 144.3)
- added REF**177: TestPoint_THTPad_D2.0mm_Drill1.0mm, TestPoint:TestPoint_THTPad_D2.0mm_Drill1.0mm, F.Cu at (132.4, 144.3)
- added REF**178: TestPoint_THTPad_D2.0mm_Drill1.0mm, TestPoint:TestPoint_THTPad_D2.0mm_Drill1.0mm, F.Cu at (135.0, 144.3)
- added REF**179: TestPoint_THTPad_D2.0mm_Drill1.0mm, TestPoint:TestPoint_THTPad_D2.0mm_Drill1.0mm, F.Cu at (137.5, 144.3)
- added REF**18: TestPoint_THTPad_D2.0mm_Drill1.0mm, TestPoint:TestPoint_THTPad_D2.0mm_Drill1.0mm, F.Cu at (124.8, 129.0)
- added REF**180: TestPoint_THTPad_D2.0mm_Drill1.0mm, TestPoint:TestPoint_THTPad_D2.0mm_Drill1.0mm, F.Cu at (140.0, 144.3)
- added REF**181: TestPoint_THTPad_D2.0mm_Drill1.0mm, TestPoint:TestPoint_THTPad_D2.0mm_Drill1.0mm, F.Cu at (142.6, 144.3)
- added REF**182: TestPoint_THTPad_D2.0mm_Drill1.0mm, TestPoint:TestPoint_THTPad_D2.0mm_Drill1.0mm, F.Cu at (79.1, 146.8)
- added REF**183: TestPoint_THTPad_D2.0mm_Drill1.0mm, TestPoint:TestPoint_THTPad_D2.0mm_Drill1.0mm, F.Cu at (81.6, 146.8)
- added REF**184: TestPoint_THTPad_D2.0mm_Drill1.0mm, TestPoint:TestPoint_THTPad_D2.0mm_Drill1.0mm, F.Cu at (84.2, 146.8)
- added REF**185: TestPoint_THTPad_D2.0mm_Drill1.0mm, TestPoint:TestPoint_THTPad_D2.0mm_Drill1.0mm, F.Cu at (86.7, 146.8)
- added REF**186: TestPoint_THTPad_D2.0mm_Drill1.0mm, TestPoint:TestPoint_THTPad_D2.0mm_Drill1.0mm, F.Cu at (89.2, 146.8)
- added REF**187: TestPoint_THTPad_D2.0mm_Drill1.0mm, TestPoint:TestPoint_THTPad_D2.0mm_Drill1.0mm, F.Cu at (91.8, 146.8)
- added REF**188: TestPoint_THTPad_D2.0mm_Drill1.0mm, TestPoint:TestPoint_THTPad_D2.0mm_Drill1.0mm, F.Cu at (94.3, 146.8)
- added REF**189: TestPoint_THTPad_D2.0mm_Drill1.0mm, TestPoint:TestPoint_THTPad_D2.0mm_Drill1.0mm, F.Cu at (96.9, 146.8)
- added REF**19: TestPoint_THTPad_D2.0mm_Drill1.0mm, TestPoint:TestPoint_THTPad_D2.0mm_Drill1.0mm, F.Cu at (127.3, 129.0)
- added REF**190: TestPoint_THTPad_D2.0mm_Drill1.0mm, TestPoint:TestPoint_THTPad_D2.0mm_Drill1.0mm, F.Cu at (99.4, 146.8)
- added REF**191: TestPoint_THTPad_D2.0mm_Drill1.0mm, TestPoint:TestPoint_THTPad_D2.0mm_Drill1.0mm, F.Cu at (101.9, 146.8)
- added REF**192: TestPoint_THTPad_D2.0mm_Drill1.0mm, TestPoint:TestPoint_THTPad_D2.0mm_Drill1.0mm, F.Cu at (104.5, 146.8)
- added REF**193: TestPoint_THTPad_D2.0mm_Drill1.0mm, TestPoint:TestPoint_THTPad_D2.0mm_Drill1.0mm, F.Cu at (107.0, 146.8)
- added REF**194: TestPoint_THTPad_D2.0mm_Drill1.0mm, TestPoint:TestPoint_THTPad_D2.0mm_Drill1.0mm, F.Cu at (109.6, 146.8)
- added REF**195: TestPoint_THTPad_D2.0mm_Drill1.0mm, TestPoint:TestPoint_THTPad_D2.0mm_Drill1.0mm, F.Cu at (112.1, 146.8)
- added REF**196: TestPoint_THTPad_D2.0mm_Drill1.0mm, TestPoint:TestPoint_THTPad_D2.0mm_Drill1.0mm, F.Cu at (114.6, 146.8)
- added REF**197: TestPoint_THTPad_D2.0mm_Drill1.0mm, TestPoint:TestPoint_THTPad_D2.0mm_Drill1.0mm, F.Cu at (117.2, 146.8)
- added REF**198: TestPoint_THTPad_D2.0mm_Drill1.0mm, TestPoint:TestPoint_THTPad_D2.0mm_Drill1.0mm, F.Cu at (119.7, 146.8)
- added REF**199: TestPoint_THTPad_D2.0mm_Drill1.0mm, TestPoint:TestPoint_THTPad_D2.0mm_Drill1.0mm, F.Cu at (122.3, 146.8)
- added REF**2: TestPoint_THTPad_D2.0mm_Drill1.0mm, TestPoint:TestPoint_THTPad_D2.0mm_Drill1.0mm, F.Cu at (84.2, 129.0)
- added REF**20: TestPoint_THTPad_D2.0mm_Drill1.0mm, TestPoint:TestPoint_THTPad_D2.0mm_Drill1.0mm, F.Cu at (129.9, 129.0)
- added REF**200: TestPoint_THTPad_D2.0mm_Drill1.0mm, TestPoint:TestPoint_THTPad_D2.0mm_Drill1.0mm, F.Cu at (124.8, 146.8)
- added REF**201: TestPoint_THTPad_D2.0mm_Drill1.0mm, TestPoint:TestPoint_THTPad_D2.0mm_Drill1.0mm, F.Cu at (127.3, 146.8)
- added REF**202: TestPoint_THTPad_D2.0mm_Drill1.0mm, TestPoint:TestPoint_THTPad_D2.0mm_Drill1.0mm, F.Cu at (129.9, 146.8)
- added REF**203: TestPoint_THTPad_D2.0mm_Drill1.0mm, TestPoint:TestPoint_THTPad_D2.0mm_Drill1.0mm, F.Cu at (132.4, 146.8)
- added REF**204: TestPoint_THTPad_D2.0mm_Drill1.0mm, TestPoint:TestPoint_THTPad_D2.0mm_Drill1.0mm, F.Cu at (135.0, 146.8)
- added REF**205: TestPoint_THTPad_D2.0mm_Drill1.0mm, TestPoint:TestPoint_THTPad_D2.0mm_Drill1.0mm, F.Cu at (137.5, 146.8)
- added REF**206: TestPoint_THTPad_D2.0mm_Drill1.0mm, TestPoint:TestPoint_THTPad_D2.0mm_Drill1.0mm, F.Cu at (140.0, 146.8)
- added REF**207: TestPoint_THTPad_D2.0mm_Drill1.0mm, TestPoint:TestPoint_THTPad_D2.0mm_Drill1.0mm, F.Cu at (142.6, 146.8)
- added REF**208: TestPoint_THTPad_D2.0mm_Drill1.0mm, TestPoint:TestPoint_THTPad_D2.0mm_Drill1.0mm, F.Cu at (79.1, 149.3)
- added REF**209: TestPoint_THTPad_D2.0mm_Drill1.0mm, TestPoint:TestPoint_THTPad_D2.0mm_Drill1.0mm, F.Cu at (81.6, 149.3)
- added REF**21: TestPoint_THTPad_D2.0mm_Drill1.0mm, TestPoint:TestPoint_THTPad_D2.0mm_Drill1.0mm, F.Cu at (132.4, 129.0)
- added REF**210: TestPoint_THTPad_D2.0mm_Drill1.0mm, TestPoint:TestPoint_THTPad_D2.0mm_Drill1.0mm, F.Cu at (84.2, 149.3)
- added REF**211: TestPoint_THTPad_D2.0mm_Drill1.0mm, TestPoint:TestPoint_THTPad_D2.0mm_Drill1.0mm, F.Cu at (86.7, 149.3)
- added REF**212: TestPoint_THTPad_D2.0mm_Drill1.0mm, TestPoint:TestPoint_THTPad_D2.0mm_Drill1.0mm, F.Cu at (89.2, 149.3)
- added REF**213: TestPoint_THTPad_D2.0mm_Drill1.0mm, TestPoint:TestPoint_THTPad_D2.0mm_Drill1.0mm, F.Cu at (91.8, 149.3)
- added REF**214: TestPoint_THTPad_D2.0mm_Drill1.0mm, TestPoint:TestPoint_THTPad_D2.0mm_Drill1.0mm, F.Cu at (94.3, 149.3)
- added REF**215: TestPoint_THTPad_D2.0mm_Drill1.0mm, TestPoint:TestPoint_THTPad_D2.0mm_Drill1.0mm, F.Cu at (96.9, 149.3)
- added REF**216: TestPoint_THTPad_D2.0mm_Drill1.0mm, TestPoint:TestPoint_THTPad_D2.0mm_Drill1.0mm, F.Cu at (99.4, 149.3)
- added REF**217: TestPoint_THTPad_D2.0mm_Drill1.0mm, TestPoint:TestPoint_THTPad_D2.0mm_Drill1.0mm, F.Cu at (101.9, 149.3)
- added REF**218: TestPoint_THTPad_D2.0mm_Drill1.0mm, TestPoint:TestPoint_THTPad_D2.0mm_Drill1.0mm, F.Cu at (104.5, 149.3)
- added REF**219: TestPoint_THTPad_D2.0mm_Drill1.0mm, TestPoint:TestPoint_THTPad_D2.0mm_Drill1.0mm, F.Cu at (107.0, 149.3)
- added REF**22: TestPoint_THTPad_D2.0mm_Drill1.0mm, TestPoint:TestPoint_THTPad_D2.0mm_Drill1.0mm, F.Cu at (135.0, 129.0)
- added REF**220: TestPoint_THTPad_D2.0mm_Drill1.0mm, TestPoint:TestPoint_THTPad_D2.0mm_Drill1.0mm, F.Cu at (109.6, 149.3)
- added REF**221: TestPoint_THTPad_D2.0mm_Drill1.0mm, TestPoint:TestPoint_THTPad_D2.0mm_Drill1.0mm, F.Cu at (112.1, 149.3)
- added REF**222: TestPoint_THTPad_D2.0mm_Drill1.0mm, TestPoint:TestPoint_THTPad_D2.0mm_Drill1.0mm, F.Cu at (114.6, 149.3)
- added REF**223: TestPoint_THTPad_D2.0mm_Drill1.0mm, TestPoint:TestPoint_THTPad_D2.0mm_Drill1.0mm, F.Cu at (117.2, 149.3)
- added REF**224: TestPoint_THTPad_D2.0mm_Drill1.0mm, TestPoint:TestPoint_THTPad_D2.0mm_Drill1.0mm, F.Cu at (119.7, 149.3)
- added REF**225: TestPoint_THTPad_D2.0mm_Drill1.0mm, TestPoint:TestPoint_THTPad_D2.0mm_Drill1.0mm, F.Cu at (122.3, 149.3)
- added REF**226: TestPoint_THTPad_D2.0mm_Drill1.0mm, TestPoint:TestPoint_THTPad_D2.0mm_Drill1.0mm, F.Cu at (124.8, 149.3)
- added REF**227: TestPoint_THTPad_D2.0mm_Drill1.0mm, TestPoint:TestPoint_THTPad_D2.0mm_Drill1.0mm, F.Cu at (127.3, 149.3)
- added REF**228: TestPoint_THTPad_D2.0mm_Drill1.0mm, TestPoint:TestPoint_THTPad_D2.0mm_Drill1.0mm, F.Cu at (129.9, 149.3)
- added REF**229: TestPoint_THTPad_D2.0mm_Drill1.0mm, TestPoint:TestPoint_THTPad_D2.0mm_Drill1.0mm, F.Cu at (132.4, 149.3)
- added REF**23: TestPoint_THTPad_D2.0mm_Drill1.0mm, TestPoint:TestPoint_THTPad_D2.0mm_Drill1.0mm, F.Cu at (137.5, 129.0)
- added REF**230: TestPoint_THTPad_D2.0mm_Drill1.0mm, TestPoint:TestPoint_THTPad_D2.0mm_Drill1.0mm, F.Cu at (135.0, 149.3)
- added REF**231: TestPoint_THTPad_D2.0mm_Drill1.0mm, TestPoint:TestPoint_THTPad_D2.0mm_Drill1.0mm, F.Cu at (137.5, 149.3)
- added REF**232: TestPoint_THTPad_D2.0mm_Drill1.0mm, TestPoint:TestPoint_THTPad_D2.0mm_Drill1.0mm, F.Cu at (140.0, 149.3)
- added REF**233: TestPoint_THTPad_D2.0mm_Drill1.0mm, TestPoint:TestPoint_THTPad_D2.0mm_Drill1.0mm, F.Cu at (142.6, 149.3)
- added REF**234: TestPoint_THTPad_D2.0mm_Drill1.0mm, TestPoint:TestPoint_THTPad_D2.0mm_Drill1.0mm, F.Cu at (79.1, 151.9)
- added REF**235: TestPoint_THTPad_D2.0mm_Drill1.0mm, TestPoint:TestPoint_THTPad_D2.0mm_Drill1.0mm, F.Cu at (81.6, 151.9)
- added REF**236: TestPoint_THTPad_D2.0mm_Drill1.0mm, TestPoint:TestPoint_THTPad_D2.0mm_Drill1.0mm, F.Cu at (84.2, 151.9)
- added REF**237: TestPoint_THTPad_D2.0mm_Drill1.0mm, TestPoint:TestPoint_THTPad_D2.0mm_Drill1.0mm, F.Cu at (86.7, 151.9)
- added REF**238: TestPoint_THTPad_D2.0mm_Drill1.0mm, TestPoint:TestPoint_THTPad_D2.0mm_Drill1.0mm, F.Cu at (89.2, 151.9)
- added REF**239: TestPoint_THTPad_D2.0mm_Drill1.0mm, TestPoint:TestPoint_THTPad_D2.0mm_Drill1.0mm, F.Cu at (91.8, 151.9)
- added REF**24: TestPoint_THTPad_D2.0mm_Drill1.0mm, TestPoint:TestPoint_THTPad_D2.0mm_Drill1.0mm, F.Cu at (140.0, 129.0)
- added REF**240: TestPoint_THTPad_D2.0mm_Drill1.0mm, TestPoint:TestPoint_THTPad_D2.0mm_Drill1.0mm, F.Cu at (94.3, 151.9)
- added REF**241: TestPoint_THTPad_D2.0mm_Drill1.0mm, TestPoint:TestPoint_THTPad_D2.0mm_Drill1.0mm, F.Cu at (96.9, 151.9)
- added REF**242: TestPoint_THTPad_D2.0mm_Drill1.0mm, TestPoint:TestPoint_THTPad_D2.0mm_Drill1.0mm, F.Cu at (99.4, 151.9)
- added REF**243: TestPoint_THTPad_D2.0mm_Drill1.0mm, TestPoint:TestPoint_THTPad_D2.0mm_Drill1.0mm, F.Cu at (101.9, 151.9)
- added REF**244: TestPoint_THTPad_D2.0mm_Drill1.0mm, TestPoint:TestPoint_THTPad_D2.0mm_Drill1.0mm, F.Cu at (104.5, 151.9)
- added REF**245: TestPoint_THTPad_D2.0mm_Drill1.0mm, TestPoint:TestPoint_THTPad_D2.0mm_Drill1.0mm, F.Cu at (107.0, 151.9)
- added REF**246: TestPoint_THTPad_D2.0mm_Drill1.0mm, TestPoint:TestPoint_THTPad_D2.0mm_Drill1.0mm, F.Cu at (109.6, 151.9)
- added REF**247: TestPoint_THTPad_D2.0mm_Drill1.0mm, TestPoint:TestPoint_THTPad_D2.0mm_Drill1.0mm, F.Cu at (112.1, 151.9)
- added REF**248: TestPoint_THTPad_D2.0mm_Drill1.0mm, TestPoint:TestPoint_THTPad_D2.0mm_Drill1.0mm, F.Cu at (114.6, 151.9)
- added REF**249: TestPoint_THTPad_D2.0mm_Drill1.0mm, TestPoint:TestPoint_THTPad_D2.0mm_Drill1.0mm, F.Cu at (117.2, 151.9)
- added REF**25: TestPoint_THTPad_D2.0mm_Drill1.0mm, TestPoint:TestPoint_THTPad_D2.0mm_Drill1.0mm, F.Cu at (142.6, 129.0)
- added REF**250: TestPoint_THTPad_D2.0mm_Drill1.0mm, TestPoint:TestPoint_THTPad_D2.0mm_Drill1.0mm, F.Cu at (119.7, 151.9)
- added REF**251: TestPoint_THTPad_D2.0mm_Drill1.0mm, TestPoint:TestPoint_THTPad_D2.0mm_Drill1.0mm, F.Cu at (122.3, 151.9)
- added REF**252: TestPoint_THTPad_D2.0mm_Drill1.0mm, TestPoint:TestPoint_THTPad_D2.0mm_Drill1.0mm, F.Cu at (124.8, 151.9)
- added REF**253: TestPoint_THTPad_D2.0mm_Drill1.0mm, TestPoint:TestPoint_THTPad_D2.0mm_Drill1.0mm, F.Cu at (127.3, 151.9)
- added REF**254: TestPoint_THTPad_D2.0mm_Drill1.0mm, TestPoint:TestPoint_THTPad_D2.0mm_Drill1.0mm, F.Cu at (129.9, 151.9)
- added REF**255: TestPoint_THTPad_D2.0mm_Drill1.0mm, TestPoint:TestPoint_THTPad_D2.0mm_Drill1.0mm, F.Cu at (132.4, 151.9)
- added REF**256: TestPoint_THTPad_D2.0mm_Drill1.0mm, TestPoint:TestPoint_THTPad_D2.0mm_Drill1.0mm, F.Cu at (135.0, 151.9)
- added REF**257: TestPoint_THTPad_D2.0mm_Drill1.0mm, TestPoint:TestPoint_THTPad_D2.0mm_Drill1.0mm, F.Cu at (137.5, 151.9)
- added REF**258: TestPoint_THTPad_D2.0mm_Drill1.0mm, TestPoint:TestPoint_THTPad_D2.0mm_Drill1.0mm, F.Cu at (140.0, 151.9)
- added REF**259: TestPoint_THTPad_D2.0mm_Drill1.0mm, TestPoint:TestPoint_THTPad_D2.0mm_Drill1.0mm, F.Cu at (142.6, 151.9)
- added REF**26: TestPoint_THTPad_D2.0mm_Drill1.0mm, TestPoint:TestPoint_THTPad_D2.0mm_Drill1.0mm, F.Cu at (79.1, 131.6)
- added REF**260: TestPoint_THTPad_D2.0mm_Drill1.0mm, TestPoint:TestPoint_THTPad_D2.0mm_Drill1.0mm, F.Cu at (79.1, 154.4)
- added REF**261: TestPoint_THTPad_D2.0mm_Drill1.0mm, TestPoint:TestPoint_THTPad_D2.0mm_Drill1.0mm, F.Cu at (81.6, 154.4)
- added REF**262: TestPoint_THTPad_D2.0mm_Drill1.0mm, TestPoint:TestPoint_THTPad_D2.0mm_Drill1.0mm, F.Cu at (84.2, 154.4)
- added REF**263: TestPoint_THTPad_D2.0mm_Drill1.0mm, TestPoint:TestPoint_THTPad_D2.0mm_Drill1.0mm, F.Cu at (86.7, 154.4)
- added REF**264: TestPoint_THTPad_D2.0mm_Drill1.0mm, TestPoint:TestPoint_THTPad_D2.0mm_Drill1.0mm, F.Cu at (89.2, 154.4)
- added REF**265: TestPoint_THTPad_D2.0mm_Drill1.0mm, TestPoint:TestPoint_THTPad_D2.0mm_Drill1.0mm, F.Cu at (91.8, 154.4)
- added REF**266: TestPoint_THTPad_D2.0mm_Drill1.0mm, TestPoint:TestPoint_THTPad_D2.0mm_Drill1.0mm, F.Cu at (94.3, 154.4)
- added REF**267: TestPoint_THTPad_D2.0mm_Drill1.0mm, TestPoint:TestPoint_THTPad_D2.0mm_Drill1.0mm, F.Cu at (96.9, 154.4)
- added REF**268: TestPoint_THTPad_D2.0mm_Drill1.0mm, TestPoint:TestPoint_THTPad_D2.0mm_Drill1.0mm, F.Cu at (99.4, 154.4)
- added REF**269: TestPoint_THTPad_D2.0mm_Drill1.0mm, TestPoint:TestPoint_THTPad_D2.0mm_Drill1.0mm, F.Cu at (101.9, 154.4)
- added REF**27: TestPoint_THTPad_D2.0mm_Drill1.0mm, TestPoint:TestPoint_THTPad_D2.0mm_Drill1.0mm, F.Cu at (81.6, 131.6)
- added REF**270: TestPoint_THTPad_D2.0mm_Drill1.0mm, TestPoint:TestPoint_THTPad_D2.0mm_Drill1.0mm, F.Cu at (104.5, 154.4)
- added REF**271: TestPoint_THTPad_D2.0mm_Drill1.0mm, TestPoint:TestPoint_THTPad_D2.0mm_Drill1.0mm, F.Cu at (107.0, 154.4)
- added REF**272: TestPoint_THTPad_D2.0mm_Drill1.0mm, TestPoint:TestPoint_THTPad_D2.0mm_Drill1.0mm, F.Cu at (109.6, 154.4)
- added REF**273: TestPoint_THTPad_D2.0mm_Drill1.0mm, TestPoint:TestPoint_THTPad_D2.0mm_Drill1.0mm, F.Cu at (112.1, 154.4)
- added REF**274: TestPoint_THTPad_D2.0mm_Drill1.0mm, TestPoint:TestPoint_THTPad_D2.0mm_Drill1.0mm, F.Cu at (114.6, 154.4)
- added REF**275: TestPoint_THTPad_D2.0mm_Drill1.0mm, TestPoint:TestPoint_THTPad_D2.0mm_Drill1.0mm, F.Cu at (117.2, 154.4)
- added REF**276: TestPoint_THTPad_D2.0mm_Drill1.0mm, TestPoint:TestPoint_THTPad_D2.0mm_Drill1.0mm, F.Cu at (119.7, 154.4)
- added REF**277: TestPoint_THTPad_D2.0mm_Drill1.0mm, TestPoint:TestPoint_THTPad_D2.0mm_Drill1.0mm, F.Cu at (122.3, 154.4)
- added REF**278: TestPoint_THTPad_D2.0mm_Drill1.0mm, TestPoint:TestPoint_THTPad_D2.0mm_Drill1.0mm, F.Cu at (124.8, 154.4)
- added REF**279: TestPoint_THTPad_D2.0mm_Drill1.0mm, TestPoint:TestPoint_THTPad_D2.0mm_Drill1.0mm, F.Cu at (127.3, 154.4)
- added REF**28: TestPoint_THTPad_D2.0mm_Drill1.0mm, TestPoint:TestPoint_THTPad_D2.0mm_Drill1.0mm, F.Cu at (84.2, 131.6)
- added REF**280: TestPoint_THTPad_D2.0mm_Drill1.0mm, TestPoint:TestPoint_THTPad_D2.0mm_Drill1.0mm, F.Cu at (129.9, 154.4)
- added REF**281: TestPoint_THTPad_D2.0mm_Drill1.0mm, TestPoint:TestPoint_THTPad_D2.0mm_Drill1.0mm, F.Cu at (132.4, 154.4)
- added REF**282: TestPoint_THTPad_D2.0mm_Drill1.0mm, TestPoint:TestPoint_THTPad_D2.0mm_Drill1.0mm, F.Cu at (135.0, 154.4)
- added REF**283: TestPoint_THTPad_D2.0mm_Drill1.0mm, TestPoint:TestPoint_THTPad_D2.0mm_Drill1.0mm, F.Cu at (137.5, 154.4)
- added REF**284: TestPoint_THTPad_D2.0mm_Drill1.0mm, TestPoint:TestPoint_THTPad_D2.0mm_Drill1.0mm, F.Cu at (140.0, 154.4)
- added REF**285: TestPoint_THTPad_D2.0mm_Drill1.0mm, TestPoint:TestPoint_THTPad_D2.0mm_Drill1.0mm, F.Cu at (142.6, 154.4)
- added REF**286: TestPoint_THTPad_D2.0mm_Drill1.0mm, TestPoint:TestPoint_THTPad_D2.0mm_Drill1.0mm, F.Cu at (79.1, 157.0)
- added REF**287: TestPoint_THTPad_D2.0mm_Drill1.0mm, TestPoint:TestPoint_THTPad_D2.0mm_Drill1.0mm, F.Cu at (81.6, 157.0)
- added REF**288: TestPoint_THTPad_D2.0mm_Drill1.0mm, TestPoint:TestPoint_THTPad_D2.0mm_Drill1.0mm, F.Cu at (84.2, 157.0)
- added REF**289: TestPoint_THTPad_D2.0mm_Drill1.0mm, TestPoint:TestPoint_THTPad_D2.0mm_Drill1.0mm, F.Cu at (86.7, 157.0)
- added REF**29: TestPoint_THTPad_D2.0mm_Drill1.0mm, TestPoint:TestPoint_THTPad_D2.0mm_Drill1.0mm, F.Cu at (86.7, 131.6)
- added REF**290: TestPoint_THTPad_D2.0mm_Drill1.0mm, TestPoint:TestPoint_THTPad_D2.0mm_Drill1.0mm, F.Cu at (89.2, 157.0)
- added REF**291: TestPoint_THTPad_D2.0mm_Drill1.0mm, TestPoint:TestPoint_THTPad_D2.0mm_Drill1.0mm, F.Cu at (91.8, 157.0)
- added REF**292: TestPoint_THTPad_D2.0mm_Drill1.0mm, TestPoint:TestPoint_THTPad_D2.0mm_Drill1.0mm, F.Cu at (94.3, 157.0)
- added REF**293: TestPoint_THTPad_D2.0mm_Drill1.0mm, TestPoint:TestPoint_THTPad_D2.0mm_Drill1.0mm, F.Cu at (96.9, 157.0)
- added REF**294: TestPoint_THTPad_D2.0mm_Drill1.0mm, TestPoint:TestPoint_THTPad_D2.0mm_Drill1.0mm, F.Cu at (99.4, 157.0)
- added REF**295: TestPoint_THTPad_D2.0mm_Drill1.0mm, TestPoint:TestPoint_THTPad_D2.0mm_Drill1.0mm, F.Cu at (101.9, 157.0)
- added REF**296: TestPoint_THTPad_D2.0mm_Drill1.0mm, TestPoint:TestPoint_THTPad_D2.0mm_Drill1.0mm, F.Cu at (104.5, 157.0)
- added REF**297: TestPoint_THTPad_D2.0mm_Drill1.0mm, TestPoint:TestPoint_THTPad_D2.0mm_Drill1.0mm, F.Cu at (107.0, 157.0)
- added REF**298: TestPoint_THTPad_D2.0mm_Drill1.0mm, TestPoint:TestPoint_THTPad_D2.0mm_Drill1.0mm, F.Cu at (109.6, 157.0)
- added REF**299: TestPoint_THTPad_D2.0mm_Drill1.0mm, TestPoint:TestPoint_THTPad_D2.0mm_Drill1.0mm, F.Cu at (112.1, 157.0)
- added REF**3: TestPoint_THTPad_D2.0mm_Drill1.0mm, TestPoint:TestPoint_THTPad_D2.0mm_Drill1.0mm, F.Cu at (86.7, 129.0)
- added REF**30: TestPoint_THTPad_D2.0mm_Drill1.0mm, TestPoint:TestPoint_THTPad_D2.0mm_Drill1.0mm, F.Cu at (89.2, 131.6)
- added REF**300: TestPoint_THTPad_D2.0mm_Drill1.0mm, TestPoint:TestPoint_THTPad_D2.0mm_Drill1.0mm, F.Cu at (114.6, 157.0)
- added REF**301: TestPoint_THTPad_D2.0mm_Drill1.0mm, TestPoint:TestPoint_THTPad_D2.0mm_Drill1.0mm, F.Cu at (117.2, 157.0)
- added REF**302: TestPoint_THTPad_D2.0mm_Drill1.0mm, TestPoint:TestPoint_THTPad_D2.0mm_Drill1.0mm, F.Cu at (119.7, 157.0)
- added REF**303: TestPoint_THTPad_D2.0mm_Drill1.0mm, TestPoint:TestPoint_THTPad_D2.0mm_Drill1.0mm, F.Cu at (122.3, 157.0)
- added REF**304: TestPoint_THTPad_D2.0mm_Drill1.0mm, TestPoint:TestPoint_THTPad_D2.0mm_Drill1.0mm, F.Cu at (124.8, 157.0)
- added REF**305: TestPoint_THTPad_D2.0mm_Drill1.0mm, TestPoint:TestPoint_THTPad_D2.0mm_Drill1.0mm, F.Cu at (127.3, 157.0)
- added REF**306: TestPoint_THTPad_D2.0mm_Drill1.0mm, TestPoint:TestPoint_THTPad_D2.0mm_Drill1.0mm, F.Cu at (129.9, 157.0)
- added REF**307: TestPoint_THTPad_D2.0mm_Drill1.0mm, TestPoint:TestPoint_THTPad_D2.0mm_Drill1.0mm, F.Cu at (132.4, 157.0)
- added REF**308: TestPoint_THTPad_D2.0mm_Drill1.0mm, TestPoint:TestPoint_THTPad_D2.0mm_Drill1.0mm, F.Cu at (135.0, 157.0)
- added REF**309: TestPoint_THTPad_D2.0mm_Drill1.0mm, TestPoint:TestPoint_THTPad_D2.0mm_Drill1.0mm, F.Cu at (137.5, 157.0)
- added REF**31: TestPoint_THTPad_D2.0mm_Drill1.0mm, TestPoint:TestPoint_THTPad_D2.0mm_Drill1.0mm, F.Cu at (91.8, 131.6)
- added REF**310: TestPoint_THTPad_D2.0mm_Drill1.0mm, TestPoint:TestPoint_THTPad_D2.0mm_Drill1.0mm, F.Cu at (140.0, 157.0)
- added REF**311: TestPoint_THTPad_D2.0mm_Drill1.0mm, TestPoint:TestPoint_THTPad_D2.0mm_Drill1.0mm, F.Cu at (142.6, 157.0)
- added REF**312: TestPoint_THTPad_D2.0mm_Drill1.0mm, TestPoint:TestPoint_THTPad_D2.0mm_Drill1.0mm, F.Cu at (79.1, 159.5)
- added REF**313: TestPoint_THTPad_D2.0mm_Drill1.0mm, TestPoint:TestPoint_THTPad_D2.0mm_Drill1.0mm, F.Cu at (81.6, 159.5)
- added REF**314: TestPoint_THTPad_D2.0mm_Drill1.0mm, TestPoint:TestPoint_THTPad_D2.0mm_Drill1.0mm, F.Cu at (84.2, 159.5)
- added REF**315: TestPoint_THTPad_D2.0mm_Drill1.0mm, TestPoint:TestPoint_THTPad_D2.0mm_Drill1.0mm, F.Cu at (86.7, 159.5)
- added REF**316: TestPoint_THTPad_D2.0mm_Drill1.0mm, TestPoint:TestPoint_THTPad_D2.0mm_Drill1.0mm, F.Cu at (89.2, 159.5)
- added REF**317: TestPoint_THTPad_D2.0mm_Drill1.0mm, TestPoint:TestPoint_THTPad_D2.0mm_Drill1.0mm, F.Cu at (91.8, 159.5)
- added REF**318: TestPoint_THTPad_D2.0mm_Drill1.0mm, TestPoint:TestPoint_THTPad_D2.0mm_Drill1.0mm, F.Cu at (94.3, 159.5)
- added REF**319: TestPoint_THTPad_D2.0mm_Drill1.0mm, TestPoint:TestPoint_THTPad_D2.0mm_Drill1.0mm, F.Cu at (96.9, 159.5)
- added REF**32: TestPoint_THTPad_D2.0mm_Drill1.0mm, TestPoint:TestPoint_THTPad_D2.0mm_Drill1.0mm, F.Cu at (94.3, 131.6)
- added REF**320: TestPoint_THTPad_D2.0mm_Drill1.0mm, TestPoint:TestPoint_THTPad_D2.0mm_Drill1.0mm, F.Cu at (99.4, 159.5)
- added REF**321: TestPoint_THTPad_D2.0mm_Drill1.0mm, TestPoint:TestPoint_THTPad_D2.0mm_Drill1.0mm, F.Cu at (101.9, 159.5)
- added REF**322: TestPoint_THTPad_D2.0mm_Drill1.0mm, TestPoint:TestPoint_THTPad_D2.0mm_Drill1.0mm, F.Cu at (104.5, 159.5)
- added REF**323: TestPoint_THTPad_D2.0mm_Drill1.0mm, TestPoint:TestPoint_THTPad_D2.0mm_Drill1.0mm, F.Cu at (107.0, 159.5)
- added REF**324: TestPoint_THTPad_D2.0mm_Drill1.0mm, TestPoint:TestPoint_THTPad_D2.0mm_Drill1.0mm, F.Cu at (109.6, 159.5)
- added REF**325: TestPoint_THTPad_D2.0mm_Drill1.0mm, TestPoint:TestPoint_THTPad_D2.0mm_Drill1.0mm, F.Cu at (112.1, 159.5)
- added REF**326: TestPoint_THTPad_D2.0mm_Drill1.0mm, TestPoint:TestPoint_THTPad_D2.0mm_Drill1.0mm, F.Cu at (114.6, 159.5)
- added REF**327: TestPoint_THTPad_D2.0mm_Drill1.0mm, TestPoint:TestPoint_THTPad_D2.0mm_Drill1.0mm, F.Cu at (117.2, 159.5)
- added REF**328: TestPoint_THTPad_D2.0mm_Drill1.0mm, TestPoint:TestPoint_THTPad_D2.0mm_Drill1.0mm, F.Cu at (119.7, 159.5)
- added REF**329: TestPoint_THTPad_D2.0mm_Drill1.0mm, TestPoint:TestPoint_THTPad_D2.0mm_Drill1.0mm, F.Cu at (122.3, 159.5)
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- renumbered C901 to C201, C902 to C202, C903 to C203, C904 to C204, C905 to C205, C906 to C206, C907 to C207, C908 to C208, C911 to C209, C909 to C210, C910 to C211, C912 to C212, C913 to C213, C914 to C214, C915 to C215, C916 to C216, D28 to D101, D901 to D201, D904 to D202, IO18 to IO201, IO19 to IO202, IO20 to IO203, J901 to J201, R20 to R101, R905 to R201, R903 to R202, R904 to R203, R901 to R204, R902 to R205, R906 to R206, R907 to R207, R908 to R208, SW901 to SW201, U901 to U201, U902 to U202, U903 to U203, Y901 to Y201
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Connections:
- net MODBUS_DI renamed RELAIS_0
- U201 pad 3: MODBUS_RO -> RELAIS_1
Other:
- board size 55 x 73.5 mm -> 100 x 160 mm
- board text added: "DUT"
- board text added: "Infrastructure"
- board text added: "Octoprobe Tentacle"
- board text removed: "ZENTRALE"
