File: hardware/octoprobe_kicad_v1/pcb_dezentral_cpu.kicad_sch (KiCad schematic)
At the start: 35 parts, among them J1 USB_C_Receptacle_USB2.0, SW2 SW_MEC_5E, U1 RP2040, U3 W25Q128JVS, U4 AMS1117-3.3, Y1 Crystal_GND24_Small

Commit message: cleanup pcb
Parts:
- renumbered C15 to C901, C16 to C902, C1 to C903, C2 to C904, C3 to C905, C4 to C906, C5 to C907, C6 to C908, C7 to C909, C8 to C910, C9 to C911, C10 to C912, C11 to C913, C12 to C914, C13 to C915, C14 to C916, D1 to D901, D903 to D904, J1 to J901, R1 to R901, R2 to R902, R3 to R903, R4 to R904, R6 to R905, R7 to R906, R7 to R907, R8 to R908, SW2 to SW901, U1 to U901, U4 to U902, U3 to U903, Y1 to Y901

Commit message: initial
Parts:
- renumbered C901 to C201, C902 to C202, C903 to C203, C904 to C204, C905 to C205, C906 to C206, C907 to C207, C908 to C208, C911 to C209, C909 to C210, C910 to C211, C912 to C212, C913 to C213, C914 to C214, C915 to C215, C916 to C216, D901 to D201, D904 to D202, IO18 to IO201, IO19 to IO202, IO20 to IO203, J901 to J201, R905 to R201, R903 to R202, R904 to R203, R901 to R204, R902 to R205, R906 to R206, R907 to R207, R908 to R208, SW901 to SW201, U901 to U201, U902 to U202, U903 to U203, Y901 to Y201
Connections:
- net MODBUS_DI renamed RELAIS_0
- net MODBUS_RO renamed RELAIS_1
Other:
- moved on the sheet: C203, C204, C205, C206, C207, C208, C209, C210, C211, C212, C213, C214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

Commit message: tmp
Parts:
- removed SW201: SW_MEC_5E, 00_project_library:SW_TS-1187A-B-A-B, symbol 00_project_library:SW_MEC_5E
- added C217: 10n, symbol Device:C_Polarized
- added J202: BOOT cap enable, Connector_PinHeader_2.54mm:PinHeader_1x02_P2.54mm_Vertical, symbol Connector:Conn_01x02_Pin
- added J203: BOOT Button, Connector_PinHeader_2.54mm:PinHeader_1x02_P2.54mm_Vertical, symbol Connector:Conn_01x02_Pin
- added J204: BOOT cap 2, Connector_PinHeader_2.54mm:PinHeader_1x02_P2.54mm_Vertical, symbol Connector:Conn_01x02_Pin
- added JP201, JP202: SolderJumper_2_Bridged, symbol Jumper:SolderJumper_2_Bridged
- added SW202: RESET, 00_project_library:SW_TS-1187A-B-A-B, symbol 00_project_library:SW_MEC_5E
- added TP201: Flash CS, symbol Connector:TestPoint
Connections:
- net +3V3: no longer U201.26 (RUN)
- net GND: now also C217.2, J203.1 (Pin_1), J204.1 (Pin_1), SW202.3 (K), SW202.4 (A)
- net button: now also J202.2 (Pin_2), J203.2 (Pin_2), JP202.2 (B), TP201.1
- new net: C217.1, JP201.1 (A)
- new net: J202.1 (Pin_1), J204.2 (Pin_2), JP201.2 (B), JP202.1 (A)
- new net: SW202.1, SW202.2, U201.26 (RUN)
Other:
- moved on the sheet: C201, C202, C210, C211, D201, D202, J201, R201, R204, R205, R206, R208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
