File: hardware/octoprobe_kicad_v1/pcb_dezentral_opto_relay.kicad_sch (KiCad schematic)
At the start: 9 parts, among them J301 Conn_01x02_Socket, J402 Conn_01x02_Socket, J403 Conn_01x02_Pin, U301 GAQY221S

Commit message: tmp
Parts:
- R302: value 10K -> 4k2
Changed lines of the file:
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@@
+		)
+	)
+	(text_box "Calculation of the input resistor\n\nVdiff = 3.3V - Vf = 3.3V- 1.2V = 2.1V\nI_Fon = 0.5mA\nR = 2.1V / 0.5mA = 4.2kOhm"
+		(exclude_from_sim no)
+		(at 31.75 96.52 0)
+		(size 53.34 27.94)
+		(stroke
+			(width 0)
+			(type default)
+		)
+		(fill
+			(type none)
+		)
+		(effects
+			(font
+				(size 1.27 1.27)
+			)
+			(justify left top)
 		)
 	)
@@
 			)
 		)
-		(property "Value" "10K"
+		(property "Value" "4k2"
 			(at 92.71 64.6684 90)
 			(effects
