File: hardware/octoprobe_kicad_v1/pcb_octoprobe_gnd.kicad_sch (KiCad schematic)
At the start: 4 parts, among them J801 Conn_01x02_Socket, J802 Conn_01x02_Socket, J803 Conn_01x02_Pin

Commit message: update sheet names
Other:
- company: (none) -> Hans Märki, Märki Informatik
- title: (none) -> Octoprobe
Changed lines of the file:
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@@
 	(generator_version "8.0")
 	(paper "A4")
+	(title_block
+		(title "Octoprobe")
+		(date "2024-04-24")
+		(rev "1.0")
+		(company "Hans Märki, Märki Informatik")
+		(comment 1 "The MIT License (MIT)")
+	)
 	(junction
 		(at 113.03 116.84)
@@
 		)
 		(instances
-			(project "pcb_dezentral"
+			(project "pcb_octoprobe"
 				(path "/35c47459-45a7-4753-acae-c8b47e7575e1/c4ea3607-6829-4db8-a901-90f37795c82a"
 					(reference "J801")
@@
 		)
 		(instances
-			(project "pcb_dezentral"
+			(project "pcb_octoprobe"
 				(path "/35c47459-45a7-4753-acae-c8b47e7575e1/c4ea3607-6829-4db8-a901-90f37795c82a"
 					(reference "#PWR0801")
@@
 		)
 		(instances
-			(project "pcb_dezentral"
+			(project "pcb_octoprobe"
 				(path "/35c47459-45a7-4753-acae-c8b47e7575e1/c4ea3607-6829-4db8-a901-90f37795c82a"
 					(reference "UR801")
@@
 		)
 		(instances
-			(project "pcb_dezentral"
+			(project "pcb_octoprobe"
 				(path "/35c47459-45a7-4753-acae-c8b47e7575e1/c4ea3607-6829-4db8-a901-90f37795c82a"
 					(reference "J803")
@@
 		)
 		(instances
-			(project "pcb_dezentral"
+			(project "pcb_octoprobe"
 				(path "/35c47459-45a7-4753-acae-c8b47e7575e1/c4ea3607-6829-4db8-a901-90f37795c82a"
 					(reference "J802")
