File: hardware/octoprobe_kicad_v1/pcb_octoprobe_power.kicad_sch (KiCad schematic)
At the start: 7 parts, among them J501 Conn_01x02_Socket, J502 Conn_01x02_Socket, J503 Conn_01x02_Pin

Commit message: update sheet names
Other:
- company: (none) -> Hans Märki, Märki Informatik
- title: (none) -> Octoprobe
Changed lines of the file:
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@@
 	(generator_version "8.0")
 	(paper "A4")
+	(title_block
+		(title "Octoprobe")
+		(date "2024-04-24")
+		(rev "1.0")
+		(company "Hans Märki, Märki Informatik")
+		(comment 1 "The MIT License (MIT)")
+	)
 	(junction
 		(at 104.14 101.6)
@@
 		)
 		(instances
-			(project "pcb_dezentral"
+			(project "pcb_octoprobe"
 				(path "/35c47459-45a7-4753-acae-c8b47e7575e1/3a82e9ad-9a1c-4775-bcf5-55ea8fe3a71a"
 					(reference "UR501")
@@
 		)
 		(instances
-			(project "pcb_dezentral"
+			(project "pcb_octoprobe"
 				(path "/35c47459-45a7-4753-acae-c8b47e7575e1/3a82e9ad-9a1c-4775-bcf5-55ea8fe3a71a"
 					(reference "J503")
@@
 		)
 		(instances
-			(project "pcb_dezentral"
+			(project "pcb_octoprobe"
 				(path "/35c47459-45a7-4753-acae-c8b47e7575e1/3a82e9ad-9a1c-4775-bcf5-55ea8fe3a71a"
 					(reference "J501")
@@
 		)
 		(instances
-			(project "pcb_dezentral"
+			(project "pcb_octoprobe"
 				(path "/35c47459-45a7-4753-acae-c8b47e7575e1/3a82e9ad-9a1c-4775-bcf5-55ea8fe3a71a"
 					(reference "D501")
@@
 		)
 		(instances
-			(project "pcb_dezentral"
+			(project "pcb_octoprobe"
 				(path "/35c47459-45a7-4753-acae-c8b47e7575e1/3a82e9ad-9a1c-4775-bcf5-55ea8fe3a71a"
 					(reference "J502")
@@
 		)
 		(instances
-			(project "pcb_dezentral"
+			(project "pcb_octoprobe"
 				(path "/35c47459-45a7-4753-acae-c8b47e7575e1/3a82e9ad-9a1c-4775-bcf5-55ea8fe3a71a"
 					(reference "FanQ501")
@@
 		)
 		(instances
-			(project "pcb_dezentral"
+			(project "pcb_octoprobe"
 				(path "/35c47459-45a7-4753-acae-c8b47e7575e1/3a82e9ad-9a1c-4775-bcf5-55ea8fe3a71a"
 					(reference "R501")
@@
 		)
 		(instances
-			(project "pcb_dezentral"
+			(project "pcb_octoprobe"
 				(path "/35c47459-45a7-4753-acae-c8b47e7575e1/3a82e9ad-9a1c-4775-bcf5-55ea8fe3a71a"
 					(reference "#PWR0501")
