File: hardware/octoprobe_kicad_v1/pcb_octoprobe.kicad_pcb (KiCad board)
At the start: 2 copper layers, 100 x 160 mm, 626 parts, among them J1001 Conn_01x02_Socket, J1002 Conn_01x02_Socket, J1003 Conn_01x02_Pin, J101 Conn_01x20, J102 Conn_01x20, J103 Conn_01x20, J201 USB_C_Receptacle_USB2.0, J202 BOOT cap enable, J203 BOOT Button, J204 BOOT cap 2, J301 Conn_01x02_Socket, J302 Conn_01x02_Socket, J303 Conn_01x02_Pin, J401 Conn_01x02_Socket, J402 Conn_01x02_Socket, J403 Conn_01x02_Pin, J501 Conn_01x02_Socket, J502 Conn_01x02_Socket, J503 Conn_01x02_Pin, J601 Conn_01x02_Socket, J602 Conn_01x02_Socket, J603 Conn_01x02_Pin, J701 Conn_01x02_Socket, J702 Conn_01x02_Socket, J703 Conn_01x02_Pin, J801 Conn_01x02_Socket, J802 Conn_01x02_Socket, J803 Conn_01x02_Pin, J901 Conn_01x02_Socket, J902 Conn_01x02_Socket, J903 Conn_01x02_Pin, SW202 RESET, U1001 GAQY221S, U201 RP2040, U202 AMS1117-3.3, U203 W25Q128JVS, U301 GAQY221S, U401 GAQY221S, U701 GAQY221S, U901 GAQY221S, Y201 Crystal_GND24_Small

Commit message: Relay
Parts:
- removed D1001, D901: LED WHITE, 00_project_library:LED_0603_1608Metric
- removed FanQ501, FanQ601: NMOS, Package_TO_SOT_SMD:SOT-23
- removed J1001, J1002, J301, J302, J401, J402, J501, J502, J601, J602, J701, J702, J801, J802, J901, J902: Conn_01x02_Socket, Connector_PinSocket_2.54mm:PinSocket_1x02_P2.54mm_Vertical
- removed J1003, J303, J403, J503, J603, J703, J803, J903: Conn_01x02_Pin, Connector_PinHeader_2.54mm:PinHeader_1x02_P2.54mm_Vertical
- removed R1001, R901: 1k, Resistor_SMD:R_0402_1005Metric_Pad0.72x0.64mm_HandSolder
- removed R1002, R902: 4k2, Resistor_SMD:R_0402_1005Metric_Pad0.72x0.64mm_HandSolder
- removed U1001, U901: GAQY221S, Package_SO:SOP-4_3.8x4.1mm_P2.54mm
- removed UR1001: Relay 5, 00_project_library:opctoprobe_relay
- removed UR101, UR801: GND, 00_project_library:opctoprobe_relay
- removed UR901: Relay 4, 00_project_library:opctoprobe_relay
- added J104: Conn_01x20, 00_project_library:PinSocket_2x20_P2.54mm_Vertical-mirrored, F.Cu at (114.6, 80.8)
- added J105: Conn_01x20, 00_project_library:PinSocket_2x20_P2.54mm_Vertical-mirrored-bare, F.Cu at (114.6, 88.4)
- added R502: 4k2, Resistor_SMD:R_0402_1005Metric_Pad0.72x0.64mm_HandSolder, F.Cu at (142.5, 63.5)
- added R602: 4k2, Resistor_SMD:R_0402_1005Metric_Pad0.72x0.64mm_HandSolder, F.Cu at (147.5, 63.5)
- added U501: GAQY221S, Package_SO:SOP-4_3.8x4.1mm_P2.54mm, F.Cu at (141.4, 68.8)
- added U601: GAQY221S, Package_SO:SOP-4_3.8x4.1mm_P2.54mm, F.Cu at (146.5, 68.8)
- D501, D601: value RED -> LED WHITE
- R501, R601: value 470R -> 1k
- UR301: value Relay 1 -> 1
- UR401: value Relay 2 -> 2
- UR501: value 3V3 -> 3
- UR601: value 5V -> 4
- UR701: value Relay 3 -> 5
- moved D501 47.0 mm to (141.3, 101.0)
- moved D601 42.8 mm to (146.4, 101.0)
- moved R501 42.7 mm to (140.5, 63.5), turned to 90 degrees
- moved UR501 42.3 mm to (138.8, 102.3)
- moved R601 38.1 mm to (145.6, 63.5), turned to 90 degrees
- moved UR601 37.2 mm to (143.9, 102.3)
- moved D301 27.0 mm to (131.2, 101.1)
- moved D701 26.9 mm to (151.5, 101.0)
- moved D401 25.6 mm to (136.2, 101.0)
- moved R301 19.7 mm to (130.4, 63.5), turned to 90 degrees
- moved R701 19.6 mm to (150.7, 63.5), turned to 90 degrees
- moved R302 18.4 mm to (132.3, 63.5), turned to -90 degrees
- moved R702 18.3 mm to (152.6, 63.5), turned to -90 degrees
- moved U301 18.1 mm to (131.3, 68.8), turned to -90 degrees
- moved U701 18.0 mm to (151.6, 68.8), turned to -90 degrees
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Connections:
- D501 pad 1: Net-(D501-K) -> GND
- D601 pad 1: Net-(D601-K) -> GND
- R501 pad 1: Net-(D501-K) -> Net-(D501-A)
- R501 pad 2: DUT_3V3 -> RELAIS_3
- R601 pad 1: Net-(D601-K) -> Net-(D601-A)
- R601 pad 2: DUT_5V -> /Relay 4/RELAY_IN
- R701 pad 2: RELAIS_3 -> /Relay 5/RELAY_IN
- R702 pad 1: RELAIS_3 -> /Relay 5/RELAY_IN
- U301 pad 3: Net-(J301-Pin_2) -> /Relay 1/RELAY_OUT_A
- U301 pad 4: Net-(J301-Pin_1) -> /Relay 1/RELAY_OUT_B
- U401 pad 3: Net-(J401-Pin_2) -> /Relay 2/RELAY_OUT_A
- U401 pad 4: Net-(J401-Pin_1) -> /Relay 2/RELAY_OUT_B
- U701 pad 3: Net-(J701-Pin_2) -> /Relay 5/RELAY_OUT_A
- U701 pad 4: Net-(J701-Pin_1) -> /Relay 5/RELAY_OUT_B
Routing:
- net +3V3: track 104.1 -> 124.4 mm
- net +5V: track 10.5 -> 30.8 mm
- net GND: track 48.0 -> 68.3 mm
- net Net-(J104-Pin_39): track 0.00 -> 10.2 mm
- net Net-(J104-Pin_37): track 0.00 -> 10.2 mm
- net Net-(J104-Pin_35): track 0.00 -> 10.2 mm
- net Net-(J104-Pin_33): track 0.00 -> 10.2 mm
- net /Relay 5/RELAY_OUT_B: track 0.00 -> 10.2 mm
- net /Relay 5/RELAY_OUT_A: track 0.00 -> 10.2 mm
- net /Relay 4/RELAY_OUT_B: track 0.00 -> 10.2 mm
- net /Relay 4/RELAY_OUT_A: track 0.00 -> 10.2 mm
- net /Relay 3/RELAY_OUT_B: track 0.00 -> 10.2 mm
- net /Relay 3/RELAY_OUT_A: track 0.00 -> 10.2 mm
- net /Relay 2/RELAY_OUT_B: track 0.00 -> 10.2 mm
- net /Relay 2/RELAY_OUT_A: track 0.00 -> 10.2 mm
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Other:
- board text added: "3V3"
- board text added: "5V"

Commit message: Improve PCB
Parts:
- removed C101: 100n 50V, Diode_SMD:D_0805_2012Metric
- added BP201: GPIO12, 00_project_library:octoprobe_breakout_label, F.Cu at (152.7, 47.7)
- added BP202: GPIO13, 00_project_library:octoprobe_breakout_label, F.Cu at (152.7, 45.2)
- added BP203: GPIO14, 00_project_library:octoprobe_breakout_label, F.Cu at (152.7, 42.7)
- added BP204: GPIO15, 00_project_library:octoprobe_breakout_label, F.Cu at (152.7, 40.1)
- added BP205: GPIO9, 00_project_library:octoprobe_breakout_label, F.Cu at (152.7, 55.4)
- added BP206: GPIO10, 00_project_library:octoprobe_breakout_label, F.Cu at (152.7, 52.8)
- added BP207: GPIO12, 00_project_library:octoprobe_breakout_label, F.Cu at (152.7, 50.3)
- moved D101 81.0 mm to (80.5, 91.5), turned to 0 degrees
- moved J202 65.3 mm to (113.4, 50.3)
- moved J203 63.2 mm to (115.9, 50.3)
- moved J204 61.1 mm to (118.5, 50.3)
- moved R210 58.1 mm to (122.3, 52.8)
- moved R209 58.0 mm to (122.3, 50.3)
- moved R201 57.0 mm to (91.5, 47.0), turned to 90 degrees
- moved SW202 47.7 mm to (80.9, 96.7)
- moved D201 32.9 mm to (80.5, 88.8), turned to 0 degrees
- moved R101 19.4 mm to (126.3, 45.6), turned to 0 degrees
- moved R206 13.8 mm to (114.0, 55.4), turned to 180 degrees
- moved R402 4.79 mm to (141.4, 66.0)
- moved R602 4.79 mm to (151.6, 66.0)
- moved R302 4.79 mm to (136.4, 66.0)
- moved R502 4.79 mm to (146.5, 66.0)
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Connections:
- D101 pad 1: Net-(D101-K) -> GND
- D101 pad 2: ZENTRALE_LED -> Net-(D101-A)
- D201 pad 1: Net-(D201-K) -> GND
- D201 pad 2: +3V3 -> Net-(D201-A)
- J101 pad 1: unconnected-(J101-Pin_1-Pad1) -> GND
- J101 pad 10: unconnected-(J101-Pin_10-Pad10) -> Net-(J101-Pin_10)
- J101 pad 11: unconnected-(J101-Pin_11-Pad11) -> Net-(J101-Pin_11)
- J101 pad 12: unconnected-(J101-Pin_12-Pad12) -> Net-(J101-Pin_11)
- J101 pad 13: unconnected-(J101-Pin_13-Pad13) -> Net-(J101-Pin_13)
- J101 pad 14: unconnected-(J101-Pin_14-Pad14) -> Net-(J101-Pin_13)
- J101 pad 15: unconnected-(J101-Pin_15-Pad15) -> Net-(J101-Pin_15)
- J101 pad 16: unconnected-(J101-Pin_16-Pad16) -> Net-(J101-Pin_15)
- J101 pad 17: unconnected-(J101-Pin_17-Pad17) -> Net-(J101-Pin_17)
- J101 pad 18: unconnected-(J101-Pin_18-Pad18) -> Net-(J101-Pin_17)
- J101 pad 19: unconnected-(J101-Pin_19-Pad19) -> Net-(J101-Pin_19)
- J101 pad 2: unconnected-(J101-Pin_2-Pad2) -> GND
- J101 pad 20: unconnected-(J101-Pin_20-Pad20) -> Net-(J101-Pin_19)
- J101 pad 21: unconnected-(J101-Pin_21-Pad21) -> Net-(J101-Pin_21)
- J101 pad 22: unconnected-(J101-Pin_22-Pad22) -> Net-(J101-Pin_21)
- J101 pad 23: unconnected-(J101-Pin_23-Pad23) -> Net-(J101-Pin_23)
- J101 pad 24: unconnected-(J101-Pin_24-Pad24) -> Net-(J101-Pin_23)
- J101 pad 25: unconnected-(J101-Pin_25-Pad25) -> Net-(J101-Pin_25)
- J101 pad 26: unconnected-(J101-Pin_26-Pad26) -> Net-(J101-Pin_25)
- J101 pad 27: unconnected-(J101-Pin_27-Pad27) -> Net-(J101-Pin_27)
- J101 pad 28: unconnected-(J101-Pin_28-Pad28) -> Net-(J101-Pin_27)
- J101 pad 29: unconnected-(J101-Pin_29-Pad29) -> Net-(J101-Pin_29)
- J101 pad 3: unconnected-(J101-Pin_3-Pad3) -> GND
- J101 pad 30: unconnected-(J101-Pin_30-Pad30) -> Net-(J101-Pin_29)
- J101 pad 31: unconnected-(J101-Pin_31-Pad31) -> Net-(J101-Pin_31)
- J101 pad 32: unconnected-(J101-Pin_32-Pad32) -> Net-(J101-Pin_31)
- J101 pad 33: unconnected-(J101-Pin_33-Pad33) -> Net-(J101-Pin_33)
- J101 pad 34: unconnected-(J101-Pin_34-Pad34) -> Net-(J101-Pin_33)
- J101 pad 35: unconnected-(J101-Pin_35-Pad35) -> Net-(J101-Pin_35)
- J101 pad 36: unconnected-(J101-Pin_36-Pad36) -> Net-(J101-Pin_35)
- J101 pad 37: unconnected-(J101-Pin_37-Pad37) -> GND
- J101 pad 38: unconnected-(J101-Pin_38-Pad38) -> GND
- J101 pad 39: unconnected-(J101-Pin_39-Pad39) -> GND
- J101 pad 4: unconnected-(J101-Pin_4-Pad4) -> GND
- J101 pad 40: unconnected-(J101-Pin_40-Pad40) -> GND
- J101 pad 5: unconnected-(J101-Pin_5-Pad5) -> Net-(J101-Pin_5)
- J101 pad 6: unconnected-(J101-Pin_6-Pad6) -> Net-(J101-Pin_5)
- J101 pad 7: unconnected-(J101-Pin_7-Pad7) -> Net-(J101-Pin_7)
- J101 pad 8: unconnected-(J101-Pin_8-Pad8) -> Net-(J101-Pin_7)
- J101 pad 9: unconnected-(J101-Pin_9-Pad9) -> Net-(J101-Pin_10)
- J102 pad 1: unconnected-(J102-Pin_1-Pad1) -> GND
- J102 pad 10: unconnected-(J102-Pin_10-Pad10) -> Net-(J101-Pin_10)
- J102 pad 11: unconnected-(J102-Pin_11-Pad11) -> Net-(J101-Pin_11)
- J102 pad 12: unconnected-(J102-Pin_12-Pad12) -> Net-(J101-Pin_11)
- J102 pad 13: unconnected-(J102-Pin_13-Pad13) -> Net-(J101-Pin_13)
- J102 pad 14: unconnected-(J102-Pin_14-Pad14) -> Net-(J101-Pin_13)
- J102 pad 15: unconnected-(J102-Pin_15-Pad15) -> Net-(J101-Pin_15)
- J102 pad 16: unconnected-(J102-Pin_16-Pad16) -> Net-(J101-Pin_15)
- J102 pad 17: unconnected-(J102-Pin_17-Pad17) -> Net-(J101-Pin_17)
- J102 pad 18: unconnected-(J102-Pin_18-Pad18) -> Net-(J101-Pin_17)
- J102 pad 19: unconnected-(J102-Pin_19-Pad19) -> Net-(J101-Pin_19)
- J102 pad 2: unconnected-(J102-Pin_2-Pad2) -> GND
- J102 pad 20: unconnected-(J102-Pin_20-Pad20) -> Net-(J101-Pin_19)
- J102 pad 21: unconnected-(J102-Pin_21-Pad21) -> Net-(J101-Pin_21)
- J102 pad 22: unconnected-(J102-Pin_22-Pad22) -> Net-(J101-Pin_21)
- J102 pad 23: unconnected-(J102-Pin_23-Pad23) -> Net-(J101-Pin_23)
- J102 pad 24: unconnected-(J102-Pin_24-Pad24) -> Net-(J101-Pin_23)
- J102 pad 25: unconnected-(J102-Pin_25-Pad25) -> Net-(J101-Pin_25)
- J102 pad 26: unconnected-(J102-Pin_26-Pad26) -> Net-(J101-Pin_25)
- J102 pad 27: unconnected-(J102-Pin_27-Pad27) -> Net-(J101-Pin_27)
- J102 pad 28: unconnected-(J102-Pin_28-Pad28) -> Net-(J101-Pin_27)
- J102 pad 29: unconnected-(J102-Pin_29-Pad29) -> Net-(J101-Pin_29)
- J102 pad 3: unconnected-(J102-Pin_3-Pad3) -> GND
- J102 pad 30: unconnected-(J102-Pin_30-Pad30) -> Net-(J101-Pin_29)
- J102 pad 31: unconnected-(J102-Pin_31-Pad31) -> Net-(J101-Pin_31)
- J102 pad 32: unconnected-(J102-Pin_32-Pad32) -> Net-(J101-Pin_31)
- J102 pad 33: unconnected-(J102-Pin_33-Pad33) -> Net-(J101-Pin_33)
- J102 pad 34: unconnected-(J102-Pin_34-Pad34) -> Net-(J101-Pin_33)
- J102 pad 35: unconnected-(J102-Pin_35-Pad35) -> Net-(J101-Pin_35)
- J102 pad 36: unconnected-(J102-Pin_36-Pad36) -> Net-(J101-Pin_35)
- J102 pad 37: unconnected-(J102-Pin_37-Pad37) -> GND
- J102 pad 38: unconnected-(J102-Pin_38-Pad38) -> GND
- J102 pad 39: unconnected-(J102-Pin_39-Pad39) -> GND
- J102 pad 4: unconnected-(J102-Pin_4-Pad4) -> GND
- J102 pad 40: unconnected-(J102-Pin_40-Pad40) -> GND
- J102 pad 5: unconnected-(J102-Pin_5-Pad5) -> Net-(J101-Pin_5)
- J102 pad 6: unconnected-(J102-Pin_6-Pad6) -> Net-(J101-Pin_5)
- J102 pad 7: unconnected-(J102-Pin_7-Pad7) -> Net-(J101-Pin_7)
- J102 pad 8: unconnected-(J102-Pin_8-Pad8) -> Net-(J101-Pin_7)
- J102 pad 9: unconnected-(J102-Pin_9-Pad9) -> Net-(J101-Pin_10)
- J103 pad 1: unconnected-(J103-Pin_1-Pad1) -> GND
- J103 pad 10: unconnected-(J103-Pin_10-Pad10) -> Net-(J101-Pin_10)
- J103 pad 11: unconnected-(J103-Pin_11-Pad11) -> Net-(J101-Pin_11)
- J103 pad 12: unconnected-(J103-Pin_12-Pad12) -> Net-(J101-Pin_11)
- J103 pad 13: unconnected-(J103-Pin_13-Pad13) -> Net-(J101-Pin_13)
- J103 pad 14: unconnected-(J103-Pin_14-Pad14) -> Net-(J101-Pin_13)
- J103 pad 15: unconnected-(J103-Pin_15-Pad15) -> Net-(J101-Pin_15)
- J103 pad 16: unconnected-(J103-Pin_16-Pad16) -> Net-(J101-Pin_15)
- J103 pad 17: unconnected-(J103-Pin_17-Pad17) -> Net-(J101-Pin_17)
- J103 pad 18: unconnected-(J103-Pin_18-Pad18) -> Net-(J101-Pin_17)
- J103 pad 19: unconnected-(J103-Pin_19-Pad19) -> Net-(J101-Pin_19)
- J103 pad 2: unconnected-(J103-Pin_2-Pad2) -> GND
- J103 pad 20: unconnected-(J103-Pin_20-Pad20) -> Net-(J101-Pin_19)
- J103 pad 21: unconnected-(J103-Pin_21-Pad21) -> Net-(J101-Pin_21)
- J103 pad 22: unconnected-(J103-Pin_22-Pad22) -> Net-(J101-Pin_21)
- J103 pad 23: unconnected-(J103-Pin_23-Pad23) -> Net-(J101-Pin_23)
- J103 pad 24: unconnected-(J103-Pin_24-Pad24) -> Net-(J101-Pin_23)
- J103 pad 25: unconnected-(J103-Pin_25-Pad25) -> Net-(J101-Pin_25)
- J103 pad 26: unconnected-(J103-Pin_26-Pad26) -> Net-(J101-Pin_25)
- J103 pad 27: unconnected-(J103-Pin_27-Pad27) -> Net-(J101-Pin_27)
- J103 pad 28: unconnected-(J103-Pin_28-Pad28) -> Net-(J101-Pin_27)
- J103 pad 29: unconnected-(J103-Pin_29-Pad29) -> Net-(J101-Pin_29)
- J103 pad 3: unconnected-(J103-Pin_3-Pad3) -> GND
- J103 pad 30: unconnected-(J103-Pin_30-Pad30) -> Net-(J101-Pin_29)
- J103 pad 31: unconnected-(J103-Pin_31-Pad31) -> Net-(J101-Pin_31)
- J103 pad 32: unconnected-(J103-Pin_32-Pad32) -> Net-(J101-Pin_31)
- J103 pad 33: unconnected-(J103-Pin_33-Pad33) -> Net-(J101-Pin_33)
- J103 pad 34: unconnected-(J103-Pin_34-Pad34) -> Net-(J101-Pin_33)
- J103 pad 35: unconnected-(J103-Pin_35-Pad35) -> Net-(J101-Pin_35)
- J103 pad 36: unconnected-(J103-Pin_36-Pad36) -> Net-(J101-Pin_35)
- J103 pad 37: unconnected-(J103-Pin_37-Pad37) -> GND
- J103 pad 38: unconnected-(J103-Pin_38-Pad38) -> GND
- J103 pad 39: unconnected-(J103-Pin_39-Pad39) -> GND
- J103 pad 4: unconnected-(J103-Pin_4-Pad4) -> GND
- J103 pad 40: unconnected-(J103-Pin_40-Pad40) -> GND
- J103 pad 5: unconnected-(J103-Pin_5-Pad5) -> Net-(J101-Pin_5)
- J103 pad 6: unconnected-(J103-Pin_6-Pad6) -> Net-(J101-Pin_5)
- J103 pad 7: unconnected-(J103-Pin_7-Pad7) -> Net-(J101-Pin_7)
- J103 pad 8: unconnected-(J103-Pin_8-Pad8) -> Net-(J101-Pin_7)
- J103 pad 9: unconnected-(J103-Pin_9-Pad9) -> Net-(J101-Pin_10)
- R101 pad 1: GND -> Net-(D101-A)
- R101 pad 2: Net-(D101-K) -> ACTIVE_LED
- R201 pad 1: GND -> Net-(D201-A)
- R201 pad 2: Net-(D201-K) -> +3V3
- R601 pad 2: /Relay 4/RELAY_IN -> RELAIS_4
- R602 pad 1: /Relay 4/RELAY_IN -> RELAIS_4
- R701 pad 2: /Relay 5/RELAY_IN -> RELAIS_5
- R702 pad 1: /Relay 5/RELAY_IN -> RELAIS_5
- U201 pad 11: unconnected-(U201-GPIO8-Pad11) -> RELAIS_5
- U201 pad 12: unconnected-(U201-GPIO9-Pad12) -> Net-(U201-GPIO9)
- U201 pad 13: unconnected-(U201-GPIO10-Pad13) -> Net-(U201-GPIO10)
- U201 pad 14: unconnected-(U201-GPIO11-Pad14) -> Net-(U201-GPIO11)
- U201 pad 15: unconnected-(U201-GPIO12-Pad15) -> Net-(U201-GPIO12)
- U201 pad 16: unconnected-(U201-GPIO13-Pad16) -> Net-(U201-GPIO13)
- U201 pad 17: unconnected-(U201-GPIO14-Pad17) -> Net-(U201-GPIO14)
- U201 pad 18: unconnected-(U201-GPIO15-Pad18) -> Net-(U201-GPIO15)
- U201 pad 2: RELAIS_0 -> ACTIVE_LED
- U201 pad 34: ds_7 -> unconnected-(U201-GPIO22-Pad34)
- U201 pad 35: ds_6 -> unconnected-(U201-GPIO23-Pad35)
- U201 pad 36: ds_5 -> unconnected-(U201-GPIO24-Pad36)
- U201 pad 37: ds_4 -> unconnected-(U201-GPIO25-Pad37)
- U201 pad 38: ds_3 -> unconnected-(U201-GPIO26/ADC0-Pad38)
- U201 pad 39: ds_2 -> unconnected-(U201-GPIO27/ADC1-Pad39)
- U201 pad 4: MODBUS_DE -> RELAIS_2
- U201 pad 40: ds_1 -> unconnected-(U201-GPIO28/ADC2-Pad40)
- U201 pad 41: ds_0 -> unconnected-(U201-GPIO29/ADC3-Pad41)
- U201 pad 5: rel -> RELAIS_3
- U201 pad 6: button -> RELAIS_4
- U201 pad 8: ZENTRALE_LED -> unconnected-(U201-GPIO6-Pad8)
Routing:
- net Net-(U201-RUN): track 0.00 -> 79.3 mm, vias 0 -> 2
- net Net-(D101-A): track 0.00 -> 71.9 mm, vias 0 -> 2
- net +5V: track 30.8 -> 95.9 mm, vias 0 -> 2
- net +3V3: track 124.4 -> 177.1 mm
- net Net-(D201-A): track 0.00 -> 47.0 mm
- net Net-(D601-A): track 0.00 -> 37.9 mm
- net Net-(D701-A): track 0.00 -> 37.9 mm
- net Net-(D401-A): track 0.00 -> 37.9 mm
- net Net-(D501-A): track 0.00 -> 37.9 mm
- net Net-(D301-A): track 0.00 -> 37.9 mm
- net RELAIS_5: track 0.00 -> 34.0 mm
- net RELAIS_4: track 0.00 -> 32.2 mm
- net RELAIS_3: track 0.00 -> 30.2 mm
- net RELAIS_2: track 0.00 -> 28.3 mm
- net RELAIS_1: track 0.00 -> 26.3 mm
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Other:
- board text added: "Active"
- board text added: "Power"
- board text added: "Reset"
- board text removed: "PWR"

Commit message: v1 rc1
Parts:
- added BP208: Flash CS, 00_project_library:octoprobe_breakout_label, F.Cu at (120.0, 45.6)
- added C217: 10uF / 25V, Capacitor_SMD:C_0805_2012Metric, F.Cu at (122.2, 56.2)
- R301, R401, R501, R601, R701: footprint Resistor_SMD:R_0402_1005Metric_Pad0.72x0.64mm_HandSolder -> Resistor_SMD:R_0402_1005Metric
- R302, R402, R502, R602, R702: value 4k2 -> 3k9; footprint Resistor_SMD:R_0402_1005Metric_Pad0.72x0.64mm_HandSolder -> Resistor_SMD:R_0402_1005Metric
- moved R205 5.26 mm to (104.6, 42.8), turned to 0 degrees
- moved R101 2.81 mm to (128.2, 47.7), turned to 90 degrees
- moved R204 1.47 mm to (107.2, 42.8)
- moved R209 0.99 mm to (122.3, 49.3)
- moved C203 0.24 mm to (125.0, 40.0)
Connections:
- H101 pad 1: (no net) -> GND
- H102 pad 1: (no net) -> GND
- H103 pad 1: (no net) -> GND
- H104 pad 1: (no net) -> GND
Routing:
- net Net-(C217-Pad1): track 0.00 -> 3.87 mm
- net Net-(D101-A): track 71.9 -> 69.7 mm
- net /cpu/QSPI_SS: track 35.1 -> 33.0 mm
- net Net-(J201-CC1): track 2.86 -> 4.57 mm
- net Net-(J201-CC2): track 6.13 -> 4.70 mm
- net /cpu/USB_D+: track 29.6 -> 28.3 mm
- net /cpu/USB_D-: track 26.6 -> 25.4 mm
- net Net-(J202-Pin_1): track 12.3 -> 13.3 mm
- net ACTIVE_LED: track 2.83 -> 3.78 mm
- net Net-(J203-Pin_2): track 3.10 -> 3.65 mm
