File: hardware/octoprobe_kicad_v1/pcb_octoprobe_cpu.kicad_sch (KiCad schematic)
At the start: 42 parts, among them J201 USB_C_Receptacle_USB2.0, J202 BOOT cap enable, J203 BOOT Button, J204 BOOT cap 2, SW202 RESET, U201 RP2040, U202 AMS1117-3.3, U203 W25Q128JVS, Y201 Crystal_GND24_Small

Commit message: update sheet names
Other:
- company: (none) -> Hans Märki, Märki Informatik
- title: CPU -> Octoprobe

Commit message: Breakout Board
Parts:
- removed JP201, JP202: SolderJumper_2_Bridged, symbol Jumper:SolderJumper_2_Bridged
- added R209, R210: 0, Resistor_SMD:R_0805_2012Metric_Pad1.20x1.40mm_HandSolder, symbol Device:R
- C217: value 10n -> 10uF / 25V; symbol Device:C_Polarized -> 00_project_library:C; JLC (none) -> C15850
Connections:
- net QSPI_SS: now also J202.2 (Pin_2), TP201.1, R209.1
- net button: no longer J202.2 (Pin_2), J203.2 (Pin_2), R206.1, TP201.1
- net at C217.1: now also R210.2
- net at J202.1 (Pin_1), J204.2 (Pin_2): now also R209.2, R210.1
- new net: J203.2 (Pin_2), R206.1
Other:
- moved on the sheet: J202, J203, J204, R206, TP201

Commit message: Breakout Board
Parts:
- removed IO201, IO202, IO203: TestPoint, TestPoint:TestPoint_Pad_D1.0mm, symbol Connector:TestPoint
Connections:
- net modbus_addr_0: no longer names the net of U201.18 (GPIO15)
- net modbus_addr_1: no longer names the net of U201.17 (GPIO14)
- net modbus_addr_2: no longer names the net of U201.16 (GPIO13)
- net modbus_addr_3: no longer names the net of U201.15 (GPIO12)
- net modbus_addr_4: no longer names the net of U201.14 (GPIO11)
- net modbus_addr_5: no longer names the net of U201.13 (GPIO10)
- net modbus_addr_6: no longer names the net of U201.12 (GPIO9)
- net modbus_addr_7: no longer names the net of U201.11 (GPIO8)
- no-connect marks 9 -> 7

Commit message: Improve PCB
Parts:
- added BP201, BP207: GPIO12, 00_project_library:octoprobe_breakout_label, symbol 00_project_library:octoprobe_breakout_label
- added BP202: GPIO13, 00_project_library:octoprobe_breakout_label, symbol 00_project_library:octoprobe_breakout_label
- added BP203: GPIO14, 00_project_library:octoprobe_breakout_label, symbol 00_project_library:octoprobe_breakout_label
- added BP204: GPIO15, 00_project_library:octoprobe_breakout_label, symbol 00_project_library:octoprobe_breakout_label
- added BP205: GPIO9, 00_project_library:octoprobe_breakout_label, symbol 00_project_library:octoprobe_breakout_label
- added BP206: GPIO10, 00_project_library:octoprobe_breakout_label, symbol 00_project_library:octoprobe_breakout_label
- J202, J203, J204: now not fitted; now left out of the parts list
Connections:
- net +3V3: now also R201.2; no longer D201.2 (A)
- net GND: now also D201.1 (K); no longer R201.1
- net RELAIS_5: now reaches U201.11 (GPIO8)
- net at U201.12 (GPIO9): now also BP205.1
- net at U201.13 (GPIO10): now also BP206.1
- net at U201.14 (GPIO11): now also BP207.1
- net at U201.15 (GPIO12): now also BP201.1
- net at U201.16 (GPIO13): now also BP202.1
- net at U201.17 (GPIO14): now also BP203.1
- net at U201.18 (GPIO15): now also BP204.1
- net MODBUS_DE renamed RELAIS_2
- net RELAIS_0 renamed ACTIVE_LED
- net ZENTRALE_LED: no longer names the net of U201.8 (GPIO6)
- net button renamed RELAIS_4
- net ds_0: no longer names the net of U201.41 (GPIO29/ADC3)
- net ds_1: no longer names the net of U201.40 (GPIO28/ADC2)
- net ds_2: no longer names the net of U201.39 (GPIO27/ADC1)
- net ds_3: no longer names the net of U201.38 (GPIO26/ADC0)
- net ds_4: no longer names the net of U201.37 (GPIO25)
- net ds_5: no longer names the net of U201.36 (GPIO24)
- net ds_6: no longer names the net of U201.35 (GPIO23)
- net ds_7: no longer names the net of U201.34 (GPIO22)
- net rel renamed RELAIS_3
- new net: D201.2 (A), R201.1
- no-connect marks 7 -> 21
Other:
- moved on the sheet: D201, R201

Commit message: v1 rc1
Parts:
- removed TP201: Flash CS, symbol Connector:TestPoint
- added BP208: Flash CS, 00_project_library:octoprobe_breakout_label, symbol 00_project_library:octoprobe_breakout_label
- C217: footprint (none) -> Capacitor_SMD:C_0805_2012Metric
Connections:
- net QSPI_SS: now also BP208.1
Changed lines of the file:
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@@
 	(wire
 		(pts
-			(xy 199.39 77.47) (xy 199.39 78.74)
-		)
-		(stroke
-			(width 0)
-			(type default)
-		)
-	)
-	(wire
-		(pts
 			(xy 121.92 151.13) (xy 125.73 151.13)
 		)
@@
 	(wire
 		(pts
+			(xy 199.39 74.93) (xy 199.39 78.74)
+		)
+		(stroke
+			(width 0)
+			(type default)
+		)
+	)
+	(wire
+		(pts
 			(xy 156.21 165.1) (xy 156.21 163.83)
 		)
@@
 	)
 	(symbol
+		(lib_id "00_project_library:octoprobe_breakout_label")
+		(at 199.39 74.93 0)
+		(unit 1)
+		(exclude_from_sim no)
+		(in_bom yes)
+		(on_board yes)
+		(dnp no)
+		(property "Reference" "BP208"
+			(at 191.262 74.93 0)
+			(effects
+				(font
+					(size 1.27 1.27)
+				)
+			)
+		)
+		(property "Value" "Flash CS"
+			(at 183.388 74.93 0)
+			(effects
+				(font
+					(size 1.27 1.27)
+				)
+			)
+		)
+		(property "Footprint" "00_project_library:octoprobe_breakout_label"
+			(at 204.47 74.93 0)
+			(effects
+				(font
+					(size 1.27 1.27)
+				)
+				(hide yes)
+			)
+		)
+		(property "Datasheet" "https://www.roth-elektronik.com/de/produkte/detail/artnr/RE233-LF/category/Laborkarten+Dual+Inline"
+			(at 204.47 74.93 0)
+			(effects
+				(font
+					(size 1.27 1.27)
+				)
+				(hide yes)
+			)
+		)
+		(property "Description" "Octoprobe Prototype Board"
+			(at 199.39 74.93 0)
+			(effects
+				(font
+					(size 1.27 1.27)
+				)
+				(hide yes)
+			)
+		)
+		(pin "1"
+		)
+		(instances
+			(project "pcb_octoprobe"
+				(path "/35c47459-45a7-4753-acae-c8b47e7575e1/24d7d496-8920-4421-a637-0c9bf263a085"
+					(reference "BP208")
+					(unit 1)
+				)
+			)
+		)
+	)
+	(symbol
 		(lib_id "00_project_library:C")
 		(at 35.56 170.18 270)
@@
 			)
 		)
-		(property "Footprint" ""
+		(property "Footprint" "Capacitor_SMD:C_0805_2012Metric"
 			(at 200.3552 114.3 0)
 			(effects
@@
 					(unit 1)
 				)
-			)
-		)
-	)
-	(symbol
-		(lib_id "Connector:TestPoint")
-		(at 199.39 77.47 0)
-		(unit 1)
-		(exclude_from_sim no)
-		(in_bom yes)
-		(on_board yes)
-		(dnp no)
-		(property "Reference" "TP201"
-			(at 196.088 68.834 0)
-			(effects
-				(font
-					(size 1.27 1.27)
-				)
-				(justify left)
-			)
-		)
-		(property "Value" "Flash CS"
-			(at 196.088 71.374 0)
-			(effects
-				(font
-					(size 1.27 1.27)
-				)
-				(justify left)
-			)
-		)
-		(property "Footprint" ""
-			(at 204.47 77.47 0)
-			(effects
-				(font
-					(size 1.27 1.27)
-				)
-				(hide yes)
-			)
-		)
-		(property "Datasheet" "~"
-			(at 204.47 77.47 0)
-			(effects
-				(font
-					(size 1.27 1.27)
-				)
-				(hide yes)
-			)
-		)
-		(property "Description" "test point"
-			(at 199.39 77.47 0)
-			(effects
-				(font
-					(size 1.27 1.27)
-				)
-				(hide yes)
-			)
-		)
-		(pin "1"
-		)
-		(instances
-			(project "pcb_octoprobe"
-				(path "/35c47459-45a7-4753-acae-c8b47e7575e1/24d7d496-8920-4421-a637-0c9bf263a085"
-					(reference "TP201")
-					(unit 1)
-				)

Commit message: PCB octoprobe tentacle v1.0
Other:
- title: Octoprobe -> Octoprobe tentacle
Changed lines of the file:
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@@
 	(paper "A4")
 	(title_block
-		(title "Octoprobe")
+		(title "Octoprobe tentacle")
 		(date "2024-04-24")
 		(rev "1.0")
