File: hardware/octoprobe_kicad_v1/pcb_octoprobe_opto_relay.kicad_sch (KiCad schematic)
At the start: 9 parts, among them J301 Conn_01x02_Socket, J402 Conn_01x02_Socket, J403 Conn_01x02_Pin, U301 GAQY221S

Commit message: update sheet names
Other:
- company: (none) -> Hans Märki, Märki Informatik
- title: (none) -> Octoprobe
Changed lines of the file:
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@@
 	(generator_version "8.0")
 	(paper "A4")
+	(title_block
+		(title "Octoprobe")
+		(date "2024-04-24")
+		(rev "1.0")
+		(company "Hans Märki, Märki Informatik")
+		(comment 1 "The MIT License (MIT)")
+	)
 	(junction
 		(at 72.39 49.53)
@@
 		)
 		(instances
-			(project "pcb_dezentral"
+			(project "pcb_octoprobe"
 				(path "/35c47459-45a7-4753-acae-c8b47e7575e1/66635fca-a3f9-4b92-989f-2a94609b1714"
 					(reference "R302")
@@
 		)
 		(instances
-			(project "pcb_dezentral"
+			(project "pcb_octoprobe"
 				(path "/35c47459-45a7-4753-acae-c8b47e7575e1/c93857e2-4cdb-4a73-87ff-b2446dc3a53c"
 					(reference "J403")
@@
 		)
 		(instances
-			(project "pcb_dezentral"
+			(project "pcb_octoprobe"
 				(path "/35c47459-45a7-4753-acae-c8b47e7575e1/66635fca-a3f9-4b92-989f-2a94609b1714"
 					(reference "R301")
@@
 		)
 		(instances
-			(project "pcb_dezentral"
+			(project "pcb_octoprobe"
 				(path "/35c47459-45a7-4753-acae-c8b47e7575e1/66635fca-a3f9-4b92-989f-2a94609b1714"
 					(reference "J301")
@@
 		)
 		(instances
-			(project "pcb_dezentral"
+			(project "pcb_octoprobe"
 				(path "/35c47459-45a7-4753-acae-c8b47e7575e1/66635fca-a3f9-4b92-989f-2a94609b1714"
 					(reference "UR301")
@@
 		)
 		(instances
-			(project "pcb_dezentral"
+			(project "pcb_octoprobe"
 				(path "/35c47459-45a7-4753-acae-c8b47e7575e1/66635fca-a3f9-4b92-989f-2a94609b1714"
 					(reference "D301")
@@
 		)
 		(instances
-			(project "pcb_dezentral"
+			(project "pcb_octoprobe"
 				(path "/35c47459-45a7-4753-acae-c8b47e7575e1/c93857e2-4cdb-4a73-87ff-b2446dc3a53c"
 					(reference "J402")
@@
 		)
 		(instances
-			(project "pcb_dezentral"
+			(project "pcb_octoprobe"
 				(path "/35c47459-45a7-4753-acae-c8b47e7575e1/c93857e2-4cdb-4a73-87ff-b2446dc3a53c"
 					(reference "TP401")
@@
 		)
 		(instances
-			(project "pcb_dezentral"
+			(project "pcb_octoprobe"
 				(path "/35c47459-45a7-4753-acae-c8b47e7575e1/66635fca-a3f9-4b92-989f-2a94609b1714"
 					(reference "U301")
@@
 		)
 		(instances
-			(project "pcb_dezentral"
+			(project "pcb_octoprobe"
 				(path "/35c47459-45a7-4753-acae-c8b47e7575e1/66635fca-a3f9-4b92-989f-2a94609b1714"
 					(reference "#PWR0302")
@@
 		)
 		(instances
-			(project "pcb_dezentral"
+			(project "pcb_octoprobe"
 				(path "/35c47459-45a7-4753-acae-c8b47e7575e1/66635fca-a3f9-4b92-989f-2a94609b1714"
 					(reference "#PWR0301")

Commit message: Breakout Board
Parts:
- U301: symbol Relay_SolidState:CPC1002N -> Relay_SolidState:TLP3123
Changed lines of the file:
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@@
 	)
 	(symbol
-		(lib_id "Relay_SolidState:CPC1002N")
+		(lib_id "Relay_SolidState:TLP3123")
 		(at 104.14 67.31 0)
 		(unit 1)
@@
 			)
 		)
-		(property "Description" "Form A, Solid State Relay (Photo MOSFET) 60V, 0.7A, 0.55Ohm, SOP-4"
+		(property "Description" "Solid State Relay (Photo MOSFET) 40V, 1A, 0.1Ohm, SO-4"
 			(at 104.14 67.31 0)
 			(effects

Commit message: Relay
Parts:
- removed J301, J402: Conn_01x02_Socket, Connector_PinSocket_2.54mm:PinSocket_1x02_P2.54mm_Vertical, symbol Connector:Conn_01x02_Socket
- removed J403: Conn_01x02_Pin, Connector_PinHeader_2.54mm:PinHeader_1x02_P2.54mm_Vertical, symbol Connector:Conn_01x02_Pin
- UR301: value ${SHEETNAME} -> ${RELAIS_NUMBER}
Connections:
- net RELAY_OUT_A: now reaches U301.3
- net RELAY_OUT_B: now reaches U301.4
Other:
- moved on the sheet: UR301

Commit message: Improve PCB
Changed lines of the file:
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@@
 		(fields_autoplaced yes)
 		(property "Reference" "UR301"
-			(at 55.245 21.59 0)
+			(at 61.595 21.59 0)
 			(effects
 				(font
@@
 		)
 		(property "Value" "${RELAIS_NUMBER}"
-			(at 55.245 24.13 0)
+			(at 61.595 24.13 0)
 			(effects
 				(font
@@
 			(effects
 				(font
-					(size 0.8 0.8)
+					(size 1.27 1.27)
 				)
 				(hide yes)
@@
 			(effects
 				(font
-					(size 0.8 0.8)
-				)
-				(hide yes)
-			)
-		)
-		(property "Description" ""
+					(size 1.27 1.27)
+				)
+				(hide yes)
+			)
+		)
+		(property "Description" "Power symbol creates a global label with name \"GND\" , ground"
 			(at 109.22 50.8 0)
 			(effects
@@
 			(effects
 				(font
-					(size 0.8 0.8)
+					(size 1.27 1.27)
 				)
 				(hide yes)
@@
 			(effects
 				(font
-					(size 0.8 0.8)
-				)
-				(hide yes)
-			)
-		)
-		(property "Description" ""
+					(size 1.27 1.27)
+				)
+				(hide yes)
+			)
+		)
+		(property "Description" "Power symbol creates a global label with name \"GND\" , ground"
 			(at 93.98 69.85 0)
 			(effects

Commit message: v1 rc1
Parts:
- removed TP401: TestPoint, symbol Connector:TestPoint
- R301: footprint Resistor_SMD:R_0402_1005Metric_Pad0.72x0.64mm_HandSolder -> Resistor_SMD:R_0402_1005Metric
- R302: value 4k2 -> 3k9; footprint Resistor_SMD:R_0402_1005Metric_Pad0.72x0.64mm_HandSolder -> Resistor_SMD:R_0402_1005Metric
Changed lines of the file:
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@@
 		)
 	)
-	(text_box "Calculation of the input resistor\n\nVdiff = 3.3V - Vf = 3.3V- 1.2V = 2.1V\nI_Fon = 0.5mA\nR = 2.1V / 0.5mA = 4.2kOhm"
+	(text_box "Calculation of the input resistor\n\nVdiff = 3.3V - Vf = 3.3V- 1.2V = 2.1V\nI_Fon = 0.5mA\nR = 2.1V / 0.5mA = 4.2kOhm\n\nE12: 3.9kOhm"
 		(exclude_from_sim no)
 		(at 31.75 96.52 0)
@@
 			)
 		)
-		(property "Value" "4k2"
+		(property "Value" "3k9"
 			(at 92.71 64.6684 90)
 			(effects
@@
 			)
 		)
-		(property "Footprint" "Resistor_SMD:R_0402_1005Metric_Pad0.72x0.64mm_HandSolder"
+		(property "Footprint" "Resistor_SMD:R_0402_1005Metric"
 			(at 92.71 66.548 90)
 			(effects
@@
 			)
 		)
-		(property "Footprint" "Resistor_SMD:R_0402_1005Metric_Pad0.72x0.64mm_HandSolder"
+		(property "Footprint" "Resistor_SMD:R_0402_1005Metric"
 			(at 91.44 47.752 90)
 			(effects
@@
 					(unit 1)
 				)
-			)
-		)
-	)
-	(symbol
-		(lib_id "Connector:TestPoint")
-		(at 72.39 49.53 0)
-		(unit 1)
-		(exclude_from_sim no)
-		(in_bom yes)
-		(on_board yes)
-		(dnp no)
-		(fields_autoplaced yes)
-		(property "Reference" "TP401"
-			(at 74.93 44.9579 0)
-			(effects
-				(font
-					(size 1.27 1.27)
-				)
-				(justify left)
-			)
-		)
-		(property "Value" "TestPoint"
-			(at 74.93 47.4979 0)
-			(effects
-				(font
-					(size 1.27 1.27)
-				)
-				(justify left)
-			)
-		)
-		(property "Footprint" ""
-			(at 77.47 49.53 0)
-			(effects
-				(font
-					(size 1.27 1.27)
-				)
-				(hide yes)
-			)
-		)
-		(property "Datasheet" "~"
-			(at 77.47 49.53 0)
-			(effects
-				(font
-					(size 1.27 1.27)
-				)
-				(hide yes)
-			)
-		)
-		(property "Description" "test point"
-			(at 72.39 49.53 0)
-			(effects
-				(font
-					(size 1.27 1.27)
-				)
-				(hide yes)
-			)
-		)
-		(pin "1"
-		)
-		(instances
-			(project "pcb_octoprobe"
-				(path "/35c47459-45a7-4753-acae-c8b47e7575e1/c93857e2-4cdb-4a73-87ff-b2446dc3a53c"
-					(reference "TP401")
-					(unit 1)
-				)
-				(path "/35c47459-45a7-4753-acae-c8b47e7575e1/66635fca-a3f9-4b92-989f-2a94609b1714"
-					(reference "TP301")
-					(unit 1)
-				)
-				(path "/35c47459-45a7-4753-acae-c8b47e7575e1/11dbe9e5-d49b-44cb-87f2-d7d490f0e7d2"
-					(reference "TP501")
-					(unit 1)
-				)
-				(path "/35c47459-45a7-4753-acae-c8b47e7575e1/9f0ce1ac-0171-4d6a-8614-107d3aa07379"
-					(reference "TP601")
-					(unit 1)
-				)
-				(path "/35c47459-45a7-4753-acae-c8b47e7575e1/b1263d91-a8e6-4644-b570-390bb3eee6dd"
-					(reference "TP701")
-					(unit 1)
-				)

Commit message: PCB octoprobe tentacle v1.0
Other:
- title: Octoprobe -> Octoprobe tentacle
Changed lines of the file:
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@@
 	(paper "A4")
 	(title_block
-		(title "Octoprobe")
+		(title "Octoprobe tentacle")
 		(date "2024-04-24")
 		(rev "1.0")
