File: hardware/octoprobe_kicad_v0.3/pcb_octoprobe_power.kicad_sch (KiCad schematic)
At the start: 7 parts, among them J501 Conn_01x02_Socket, J502 Conn_01x02_Socket, J503 Conn_01x02_Pin

Commit message: PCB: Oscillator
Parts:
- UR501: footprint 00_project_library:opctoprobe_relay -> 00_project_library:octoprobe_relay; symbol 00_project_library:opctoprobe_relay -> 00_project_library:octoprobe_relay
Changed lines of the file:
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@@
 	)
 	(symbol
-		(lib_id "00_project_library:opctoprobe_relay")
+		(lib_id "00_project_library:octoprobe_relay")
 		(at 80.01 43.18 0)
 		(unit 1)
@@
 			)
 		)
-		(property "Footprint" "00_project_library:opctoprobe_relay"
+		(property "Footprint" "00_project_library:octoprobe_relay"
 			(at 80.01 43.18 0)
 			(effects
